File: TV_PLASMA/42PQ30R/y_board/y_er_up_and_sus_up.kicad_sch (KiCad schematic)
At the start: 8 parts

Commit message: Finishing Y_ER_UP and Y_SUS_UP
Parts:
- added C702, C704, C705, C707, C717, C720: C_Small, symbol Device:C_Small
- added D11, D21, D22, D701: D_Filled, symbol Device:D_Filled
- added FL701, FL702, L703: L, symbol Device:L
- added IC704: ~, symbol irf_s21850:Unknown_Transistor_Array_1
- added Q11, Q12, Q13, Q14: Q_NIGBT_GCE, symbol Device:Q_NIGBT_GCE
- added Q701: Q_NPN_BCE, symbol Device:Q_NPN_BCE
- added Q702: Q_PNP_BCE, symbol Device:Q_PNP_BCE
- added R12, R6, R705: 10k, symbol Device:R
- added R4, R5, R728, R730: 22, symbol Device:R
- added R703, R704, R708, R709, R710, R711, R713, R714: 10, symbol Device:R
- renumbered U1 to IC701
Connections:
- net Earth: now also C717.2, C720.2
- net at IC701.10 (Vob): now also R703.1
- net 15VFY_C: now reaches IC701.11 (VDDB)
- net 15VFY_C: now also IC701.16 (VDDA), C702.1, C704.1, C705.1, IC704.1 (C1), Q701.2 (C), R728.1, R730.1
- net Y_OUT: now reaches IC701.14 (GNDA)
- net Y_OUT: now also IC701.9 (GNDB), C702.2, C704.2, C705.2, D11.2 (A), D701.2 (A), IC704.2 (C2), Q11.3 (E), Q12.3 (E), Q13.3 (E), Q14.3 (E), Q702.2 (C), R12.1, R6.2, R705.2
- net at IC701.15 (Voa): now also R704.2
- new net: C707.2, D21.2 (A), D22.1 (K), D701.1 (K), Q14.2 (C)
- new net: D22.2 (A), FL701.2, FL702.2
- new net: Q701.1 (B), Q702.1 (B), R703.2
- new net: Q701.3 (E), Q702.3 (E), R12.2, R708.1, R709.1, R710.1, R711.1, R713.1, R714.1
- new net: IC704.3 (B2), IC704.5 (B1), R704.1, R705.1
- new net: IC704.4 (E1_E2), R4.2, R5.2
- new net: Q11.1 (G), R710.2, R714.2
- new net: Q12.1 (G), R709.2, R711.2
- new net: Q13.1 (G), R708.2, R713.2
- new net: Q14.1 (G), R4.1, R5.1, R6.1
- new net 15VFY_B: R728.2, R730.2
- new net ER_CON: C717.1, C720.1, L703.2
- new net ER_CON_A: FL701.1, FL702.1, L703.1
- new net VS_B: C707.1, D11.1 (K), D21.1 (K), Q11.2 (C), Q12.2 (C), Q13.2 (C)
Other:
- moved on the sheet: C701, C713, C714, IC701, R120, R701, R702, R721
