File: TV_PLASMA/42PQ30R/y_board/y_er_up_and_sus_up.kicad_sch (KiCad schematic)
At the start: 43 parts, among them Q11 Q_NIGBT_GCE, Q12 Q_NIGBT_GCE, Q13 Q_NIGBT_GCE, Q14 Q_NIGBT_GCE, Q701 Q_NPN_BCE, Q702 Q_PNP_BCE

Commit message: Finishing VSC and VY supply
Connections:
- net 15VFY_B renamed 15VYF_B
- net 15VFY_C renamed 15VYF_C
Changed lines of the file:
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@@
 		)
 	)
-	(global_label "15VFY_B"
+	(global_label "15VYF_B"
 		(shape input)
 		(at 43.18 73.66 180)
@@
 		)
 	)
-	(global_label "15VFY_C"
+	(global_label "15VYF_C"
 		(shape output)
 		(at 85.09 66.04 0)
@@
 		)
 	)
-	(global_label "15VFY_C"
+	(global_label "15VYF_C"
 		(shape input)
 		(at 176.53 107.95 0)

Commit message: Finishing 15VF, 5VF and 15V power supply
Other:
- moved on the sheet: C701, C702, C704, C705, C707, C713, C714, C717, C720, D11, D21, D22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

Commit message: Finishing Y BOARD reverse engineering. Todo: Add reverse conduction and resistence to all output/input pins and refactor Z BOARD DRC
Parts:
- renumbered R721 to R121
Other:
- note added: "Y ENERGY RECOVERY COIL"
- note added: "Y ENERGY RECOVERY UP AND Y SUS UP"
- note added: "Y_ER_UP"
- note added: "Y_SUS_UP"
Changed lines of the file:
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@@
 		)
 	)
-	(label "Y_SUS_UP"
-		(at 214.63 63.5 0)
+	(text "Y ENERGY RECOVERY UP AND Y SUS UP"
+		(exclude_from_sim no)
+		(at 156.21 19.05 0)
 		(effects
 			(font
-				(size 1.27 1.27)
-				(thickness 0.254)
+				(size 5 5)
+				(thickness 0.6)
 				(bold yes)
 				(italic yes)
-				(color 9 1 255 1)
 			)
-			(justify left bottom)
 		)
 	)
-	(label "Y ENERGY RECOVERY COIL"
-		(at 73.66 31.75 0)
+	(text "Y_SUS_UP"
+		(exclude_from_sim no)
+		(at 219.71 64.77 0)
 		(effects
 			(font
 				(size 1.27 1.27)
+				(thickness 0.254)
+				(bold yes)
+				(italic yes)
 			)
-			(justify left bottom)
 		)
 	)
-	(label "Y ENERGY RECOVERY UP AND Y SUS UP"
-		(at 220.98 21.59 180)
+	(text "Y ENERGY RECOVERY COIL"
+		(exclude_from_sim no)
+		(at 88.9 33.02 0)
 		(effects
 			(font
-				(face "KiCad Font")
-				(size 5 5)
+				(size 2 2)
 				(thickness 0.254)
 				(bold yes)
 				(italic yes)
 			)
-			(justify right bottom)
 		)
 	)
-	(label "Y_ER_UP"
-		(at 156.21 100.33 0)
+	(text "Y_ER_UP"
+		(exclude_from_sim no)
+		(at 157.48 87.63 0)
 		(effects
 			(font
@@
 				(bold yes)
 				(italic yes)
-				(color 9 1 255 1)
 			)
-			(justify left bottom)
 		)
 	)
@@
 		(on_board yes)
 		(dnp no)
-		(property "Reference" "R721"
+		(property "Reference" "R121"
 			(at 60.96 163.83 0)
 			(effects
@@
 			(project "y_board"
 				(path "/b3bc71fd-0ca0-4281-9bf5-aadd2561d695/bbf561e2-1af7-4443-94b3-0a21168454fa"
-					(reference "R721")
+					(reference "R121")
 					(unit 1)
 				)

Commit message: Update Y-Board schematics and add Y-Board top detailed information
Parts:
- C717, C720: value C_Small -> 3.3uF/250V
Changed lines of the file:
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@@
 			)
 		)
-		(property "Value" "C_Small"
-			(at 97.79 44.4562 0)
-			(effects
-				(font
-					(size 1.27 1.27)
-				)
-				(justify left)
-				(hide yes)
+		(property "Value" "3.3uF/250V"
+			(at 82.55 48.26 0)
+			(effects
+				(font
+					(size 1.27 1.27)
+				)
+				(justify left)
 			)
 		)
@@
 		(dnp no)
 		(property "Reference" "C720"
-			(at 97.79 45.72 0)
-			(effects
-				(font
-					(size 1.27 1.27)
-				)
-				(justify left)
-			)
-		)
-		(property "Value" "C_Small"
-			(at 106.68 44.4562 0)
-			(effects
-				(font
-					(size 1.27 1.27)
-				)
-				(justify left)
-				(hide yes)
-			)
-		)
+			(at 107.95 43.18 0)
+			(effects
+				(font
+					(size 1.27 1.27)
+				)
+				(justify left)
+			)
+		)
+		(property "Value" "3.3uF/250V"
+			(at 107.95 45.72 0)
+			(effects
+				(font
+					(size 1.27 1.27)
+				)
+				(justify left)
+			)
+		)

Commit message: Finishing document detailed images
Parts:
- IC701: value ~ -> ADUM123
Changed lines of the file:
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@@
 			)
 		)
-		(property "Value" "~"
-			(at 101.6 123.19 0)
+		(property "Value" "ADUM123"
+			(at 101.6 151.13 0)
 			(effects
 				(font

Commit message: Update Power transistor names
Parts:
- D11: value D_Filled -> RFU20
- D21: value D_Filled -> RF2001
- Q11, Q12, Q13: value Q_NIGBT_GCE -> 30J124
- Q14: value Q_NIGBT_GCE -> RJP4584
Changed lines of the file:
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@@
 		(on_board yes)
 		(dnp no)
-		(fields_autoplaced yes)
 		(property "Reference" "Q12"
 			(at 231.14 69.8499 0)
@@
 			)
 		)
-		(property "Value" "Q_NIGBT_GCE"
-			(at 231.14 71.1199 0)
-			(effects
-				(font
-					(size 1.27 1.27)
-				)
-				(justify left)
-				(hide yes)
+		(property "Value" "30J124"
+			(at 231.14 72.39 0)
+			(effects
+				(font
+					(size 1.27 1.27)
+				)
+				(justify left)
 			)
 		)
@@
 		(on_board yes)
 		(dnp no)
-		(fields_autoplaced yes)
 		(property "Reference" "Q13"
 			(at 207.01 69.8499 0)
@@
 			)
 		)
-		(property "Value" "Q_NIGBT_GCE"
-			(at 207.01 71.1199 0)
-			(effects
-				(font
-					(size 1.27 1.27)
-				)
-				(justify left)
-				(hide yes)
+		(property "Value" "30J124"
+			(at 207.01 72.39 0)
+			(effects
+				(font
+					(size 1.27 1.27)
+				)
+				(justify left)
 			)
 		)
@@
 		(on_board yes)
 		(dnp no)
-		(fields_autoplaced yes)
 		(property "Reference" "Q14"
-			(at 167.64 91.4399 0)
-			(effects
-				(font
-					(size 1.27 1.27)
-				)
-				(justify left)
-			)
-		)
-		(property "Value" "Q_NIGBT_GCE"
-			(at 167.64 93.9799 0)
-			(effects
-				(font
-					(size 1.27 1.27)
-				)
-				(justify left)
-				(hide yes)
+			(at 158.75 81.28 0)
+			(effects
+				(font
+					(size 1.27 1.27)
+				)
+				(justify left)
+			)
+		)
+		(property "Value" "RJP4584"
+			(at 154.94 83.82 0)
+			(effects
+				(font
+					(size 1.27 1.27)
+				)
+				(justify left)
 			)
 		)
@@
 			)
 		)
-		(property "Value" "D_Filled"
+		(property "Value" "RF2001"
 			(at 175.26 68.5799 90)
 			(effects
@@
 				)
 				(justify left)
-				(hide yes)
 			)
 		)
@@
 		(on_board yes)
 		(dnp no)
-		(fields_autoplaced yes)
 		(property "Reference" "Q11"
 			(at 252.73 68.5799 0)
@@
 			)
 		)
-		(property "Value" "Q_NIGBT_GCE"
-			(at 252.73 71.1199 0)
-			(effects
-				(font
-					(size 1.27 1.27)
-				)
-				(justify left)
-				(hide yes)
+		(property "Value" "30J124"
+			(at 251.46 72.39 0)
+			(effects
+				(font
+					(size 1.27 1.27)
+				)
+				(justify left)
 			)
 		)
@@
 			)
 		)
-		(property "Value" "D_Filled"
+		(property "Value" "RFU20"
 			(at 261.62 95.2499 90)
 			(effects
@@
 				)
 				(justify left)
-				(hide yes)
-			)
-		)
+			)
+		)
