File: TV_PLASMA/42PQ30R/y_board/y_sus_dn_and_blocking.kicad_sch (KiCad schematic)
At the start: 39 parts, among them Q15 NMOS, Q16 Q_NIGBT_GCE, Q601 NMOS, Q604 Q_PNP_BCE

Commit message: Finishing Y_ER_UP and Y_SUS_UP
Connections:
- net 15VFY_C renamed 15VFY_B
Changed lines of the file:
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@@
 		)
 	)
-	(global_label "15VFY_C"
+	(global_label "15VFY_B"
 		(shape output)
 		(at 238.76 57.15 0)
