File: TV_PLASMA/42PQ30R/y_board/y_sus_dn_and_blocking.kicad_sch (KiCad schematic)
At the start: 39 parts, among them Q15 NMOS, Q16 Q_NIGBT_GCE, Q601 NMOS, Q604 Q_PNP_BCE

Commit message: Finishing VSC and VY supply
Connections:
- net 15VFY renamed 15VYF
- net 15VFY_B renamed 15VYF_B
Changed lines of the file:
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@@
 		)
 	)
-	(global_label "15VFY_B"
+	(global_label "15VYF_B"
 		(shape output)
 		(at 238.76 57.15 0)
@@
 		)
 	)
-	(global_label "15VFY"
+	(global_label "15VYF"
 		(shape input)
 		(at 265.43 41.91 0)

Commit message: Add control input parts 2,3 of 3
Parts:
- renumbered R1 to R608
Connections:
- net BLOCKING_5V: now also C609.1, R118.1
- net at Q601.2 (G), R608.2: no longer C609.1, R118.1
Other:
- moved on the sheet: C609, R118, R608
Changed lines of the file:
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@@
 	)
 	(junction
+		(at 151.13 90.17)
+		(diameter 0)
+		(color 0 0 0 0)
+	)
+	(junction
 		(at 186.69 127)
 		(diameter 0)
@@
 	)
 	(junction
-		(at 160.02 102.87)
+		(at 151.13 102.87)
 		(diameter 0)
 		(color 0 0 0 0)
@@
 	)
 	(junction
-		(at 160.02 90.17)
-		(diameter 0)
-		(color 0 0 0 0)
-	)
-	(junction
 		(at 257.81 69.85)
 		(diameter 0)
@@
 	)
 	(junction
-		(at 152.4 90.17)
-		(diameter 0)
-		(color 0 0 0 0)
-	)
-	(junction
 		(at 246.38 144.78)
 		(diameter 0)
@@
 	(wire
 		(pts
-			(xy 152.4 90.17) (xy 152.4 88.9)
+			(xy 54.61 76.2) (xy 54.61 83.82)
 		)
 		(stroke
@@
 	(wire
 		(pts
-			(xy 54.61 76.2) (xy 54.61 83.82)
+			(xy 33.02 62.23) (xy 33.02 68.58)
 		)
 		(stroke
@@
 	(wire
 		(pts
-			(xy 33.02 62.23) (xy 33.02 68.58)
+			(xy 125.73 121.92) (xy 125.73 115.57)
 		)
 		(stroke
@@
 	(wire
 		(pts
-			(xy 125.73 121.92) (xy 125.73 115.57)
+			(xy 264.16 57.15) (xy 264.16 53.34)
 		)
 		(stroke
@@
 	(wire
 		(pts
-			(xy 264.16 57.15) (xy 264.16 53.34)
+			(xy 177.8 144.78) (xy 186.69 144.78)
 		)
 		(stroke
@@
 	(wire
 		(pts
-			(xy 177.8 144.78) (xy 186.69 144.78)
+			(xy 83.82 144.78) (xy 90.17 144.78)
 		)
 		(stroke
@@
 	(wire
 		(pts
-			(xy 83.82 144.78) (xy 90.17 144.78)
+			(xy 246.38 76.2) (xy 246.38 69.85)
 		)
 		(stroke
@@
 	(wire
 		(pts
-			(xy 246.38 76.2) (xy 246.38 69.85)
+			(xy 151.13 90.17) (xy 154.94 90.17)
 		)
 		(stroke
@@
 	(wire
 		(pts
-			(xy 166.37 90.17) (xy 160.02 90.17)
+			(xy 162.56 90.17) (xy 166.37 90.17)
 		)
 		(stroke
@@
 	(wire
 		(pts
-			(xy 152.4 74.93) (xy 139.7 74.93)
-		)
-		(stroke
-			(width 0)
-			(type default)
-		)
-	)
-	(wire
-		(pts
 			(xy 257.81 69.85) (xy 257.81 76.2)
 		)
@@
 	(wire
 		(pts
+			(xy 140.97 78.74) (xy 151.13 78.74)
+		)
+		(stroke
+			(width 0)
+			(type default)
+		)
+	)
+	(wire
+		(pts
 			(xy 44.45 144.78) (xy 44.45 139.7)
 		)
@@
 	(wire
 		(pts
+			(xy 151.13 78.74) (xy 151.13 90.17)
+		)
+		(stroke
+			(width 0)
+			(type default)
+		)
+	)
+	(wire
+		(pts
 			(xy 203.2 127) (xy 199.39 127)
 		)
@@
 	(wire
 		(pts
-			(xy 160.02 90.17) (xy 160.02 92.71)
+			(xy 151.13 90.17) (xy 151.13 92.71)
 		)
 		(stroke
@@
 	(wire
 		(pts
-			(xy 152.4 102.87) (xy 160.02 102.87)
+			(xy 143.51 102.87) (xy 151.13 102.87)
 		)
 		(stroke
@@
 	(wire
 		(pts
-			(xy 160.02 102.87) (xy 173.99 102.87)
-		)
-		(stroke
-			(width 0)
-			(type default)
-		)
-	)
-	(wire
-		(pts
-			(xy 152.4 81.28) (xy 152.4 74.93)
+			(xy 151.13 102.87) (xy 173.99 102.87)
 		)
 		(stroke
@@
 	(wire
 		(pts
-			(xy 160.02 90.17) (xy 152.4 90.17)
+			(xy 151.13 90.17) (xy 143.51 90.17)
 		)
 		(stroke
@@
 	(wire
 		(pts
-			(xy 152.4 90.17) (xy 152.4 93.98)
+			(xy 143.51 90.17) (xy 143.51 93.98)
 		)
 		(stroke
@@
 	(wire
 		(pts
-			(xy 160.02 100.33) (xy 160.02 102.87)
+			(xy 151.13 100.33) (xy 151.13 102.87)
 		)
 		(stroke
@@
 	(wire
 		(pts
-			(xy 152.4 99.06) (xy 152.4 102.87)
+			(xy 143.51 99.06) (xy 143.51 102.87)
 		)
 		(stroke
@@
 	(global_label "BLOCKING_5V"
 		(shape input)
-		(at 139.7 74.93 180)
+		(at 140.97 78.74 180)
 		(fields_autoplaced yes)
 		(effects
@@
 		)
 		(property "Intersheetrefs" "${INTERSHEET_REFS}"
-			(at 124.0752 74.93 0)
+			(at 125.3452 78.74 0)
 			(effects
 				(font
@@
 	(symbol
 		(lib_id "Device:R")
-		(at 152.4 85.09 0)
+		(at 158.75 90.17 90)
 		(unit 1)
 		(exclude_from_sim no)
@@
 		(on_board yes)
 		(dnp no)
-		(property "Reference" "R1"
-			(at 154.94 85.09 0)
+		(property "Reference" "R608"
+			(at 158.75 83.82 90)
 			(effects
 				(font
@@
 		)
 		(property "Value" "100"
-			(at 156.21 87.63 0)
+			(at 158.75 86.36 90)
 			(effects
 				(font
@@
 		)
 		(property "Footprint" ""
-			(at 150.622 85.09 90)
+			(at 158.75 91.948 90)
 			(effects
 				(font
@@
 		)
 		(property "Datasheet" "~"
-			(at 152.4 85.09 0)
+			(at 158.75 90.17 0)
 			(effects
 				(font
@@
 		)
 		(property "Description" "Resistor"
-			(at 152.4 85.09 0)
+			(at 158.75 90.17 0)
 			(effects
 				(font
@@
 			(project "y_board"
 				(path "/b3bc71fd-0ca0-4281-9bf5-aadd2561d695/b76c5e00-b7dd-4fa5-9261-12497b90aceb"
-					(reference "R1")
+					(reference "R608")
 					(unit 1)
 				)
@@
 	(symbol
 		(lib_id "Device:C_Small")
-		(at 152.4 96.52 0)
+		(at 143.51 96.52 0)
 		(unit 1)
 		(exclude_from_sim no)
@@
 		(dnp no)
 		(property "Reference" "C609"
-			(at 146.05 99.06 0)
+			(at 137.16 99.06 0)
 			(effects
 				(font
@@
 		)
 		(property "Value" "~"
-			(at 154.94 97.7962 0)
+			(at 146.05 97.7962 0)
 			(effects
 				(font
@@
 		)
 		(property "Footprint" ""
-			(at 152.4 96.52 0)
+			(at 143.51 96.52 0)
 			(effects
 				(font
@@
 		)
 		(property "Datasheet" "~"
-			(at 152.4 96.52 0)
+			(at 143.51 96.52 0)
 			(effects
 				(font
@@
 		)
 		(property "Description" "Unpolarized capacitor, small symbol"
-			(at 152.4 96.52 0)
+			(at 143.51 96.52 0)
 			(effects
 				(font
@@
 	(symbol
 		(lib_id "Device:R")
-		(at 160.02 96.52 0)
+		(at 151.13 96.52 0)
 		(unit 1)
 		(exclude_from_sim no)
@@
 		(dnp no)
 		(property "Reference" "R118"
-			(at 161.29 95.25 0)
+			(at 152.4 95.25 0)
 			(effects
 				(font
@@
 		)
 		(property "Value" "4.2k"
-			(at 161.29 97.79 0)
+			(at 152.4 97.79 0)
 			(effects
 				(font
@@
 		)
 		(property "Footprint" ""
-			(at 158.242 96.52 90)
+			(at 149.352 96.52 90)
 			(effects
 				(font
@@
 		)
 		(property "Datasheet" "~"
-			(at 160.02 96.52 0)
+			(at 151.13 96.52 0)
 			(effects
 				(font
@@
 		)
 		(property "Description" "Resistor"
-			(at 160.02 96.52 0)
+			(at 151.13 96.52 0)
 			(effects
 				(font

Commit message: Finishing Y BOARD reverse engineering. Todo: Add reverse conduction and resistence to all output/input pins and refactor Z BOARD DRC
Parts:
- IC703: value ~ -> S21850
- renumbered R740 to R540, R741 to R541, R742 to R542, R743 to R543, R614 to R611
Other:
- note added: "BLOCKING"
- note added: "Y BLOCKING AND Y SUS DOWN"
- note added: "Y_SUS_DOWN"
Changed lines of the file:
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@@
 		)
 	)
-	(label "Y_SUS_DOWN"
-		(at 127 132.08 0)
+	(text "Y_SUS_DOWN"
+		(exclude_from_sim no)
+		(at 133.35 132.08 0)
 		(effects
 			(font
@@
 				(bold yes)
 				(italic yes)
-				(color 9 1 255 1)
-			)
-			(justify left bottom)
-		)
-	)
-	(label "Y BLOCKING AND Y SUS DOWN"
-		(at 204.47 24.13 180)
-		(effects
-			(font
-				(face "KiCad Font")
-				(size 5 5)
-				(thickness 0.254)
-				(bold yes)
-				(italic yes)
-			)
-			(justify right bottom)
-		)
-	)
-	(label "BLOCKING"
-		(at 166.37 130.81 0)
+			)
+		)
+	)
+	(text "BLOCKING"
+		(exclude_from_sim no)
+		(at 170.18 130.81 0)
 		(effects
 			(font
@@
 				(bold yes)
 				(italic yes)
-				(color 9 1 255 1)
-			)
-			(justify left bottom)
+			)
+		)
+	)
+	(text "Y BLOCKING AND Y SUS DOWN"
+		(exclude_from_sim no)
+		(at 146.05 21.59 0)
+		(effects
+			(font
+				(size 5 5)
+				(thickness 0.6)
+				(bold yes)
+				(italic yes)
+			)
 		)
 	)
@@
 	)
 	(symbol
+		(lib_name "S21850_1")
+		(lib_id "irf_s21850:S21850")
+		(at 68.58 120.65 0)
+		(unit 1)
+		(exclude_from_sim no)
+		(in_bom yes)
+		(on_board yes)
+		(dnp no)
+		(property "Reference" "IC703"
+			(at 68.58 118.11 0)
+			(effects
+				(font
+					(size 1.27 1.27)
+				)
+			)
+		)
+		(property "Value" "S21850"
+			(at 68.58 118.11 0)
+			(effects
+				(font
+					(size 1.27 1.27)
+				)
+				(hide yes)
+			)
+		)
+		(property "Footprint" ""
+			(at 67.31 123.19 0)
+			(effects
+				(font
+					(size 1.27 1.27)
+				)
+				(hide yes)
+			)
+		)
+		(property "Datasheet" "https://www.alldatasheet.net/datasheet-pdf/download/578411/IRF/IRS21850SPBF.html"
+			(at 67.31 123.19 0)
+			(effects
+				(font
+					(size 1.27 1.27)
+				)
+				(hide yes)
+			)
+		)
+		(property "Description" ""
+			(at 67.31 123.19 0)
+			(effects
+				(font
+					(size 1.27 1.27)
+				)
+				(hide yes)
+			)
+		)
+		(pin "4"
+		)
+		(pin "2"
+		)
+		(pin "3"
+		)
+		(pin "1"
+		)
+		(pin "5"
+		)
+		(pin "8"
+		)
+		(pin "6"
+		)
+		(pin "7"
+		)
+		(instances
+			(project "y_board"
+				(path "/b3bc71fd-0ca0-4281-9bf5-aadd2561d695/b76c5e00-b7dd-4fa5-9261-12497b90aceb"
+					(reference "IC703")
+					(unit 1)
+				)
+			)
+		)
+	)
+	(symbol
 		(lib_id "Simulation_SPICE:NMOS")
 		(at 180.34 127 0)
@@
 		(dnp no)
 		(fields_autoplaced yes)
-		(property "Reference" "R742"
+		(property "Reference" "R542"
 			(at 57.15 71.1199 0)
 			(effects
@@
 			(project "y_board"
 				(path "/b3bc71fd-0ca0-4281-9bf5-aadd2561d695/b76c5e00-b7dd-4fa5-9261-12497b90aceb"
-					(reference "R742")
+					(reference "R542")
 					(unit 1)
 				)
@@
 		(on_board yes)
 		(dnp no)
-		(property "Reference" "R614"
+		(property "Reference" "R611"
 			(at 195.58 129.54 90)
 			(effects
@@
 			(project "y_board"
 				(path "/b3bc71fd-0ca0-4281-9bf5-aadd2561d695/b76c5e00-b7dd-4fa5-9261-12497b90aceb"
-					(reference "R614")
+					(reference "R611")
 					(unit 1)
 				)
@@
 		(dnp no)
 		(fields_autoplaced yes)
-		(property "Reference" "R741"
+		(property "Reference" "R541"
 			(at 45.72 71.1199 0)
 			(effects
@@
 			(project "y_board"
 				(path "/b3bc71fd-0ca0-4281-9bf5-aadd2561d695/b76c5e00-b7dd-4fa5-9261-12497b90aceb"
-					(reference "R741")
+					(reference "R541")
 					(unit 1)
 				)
@@
 		(dnp no)
 		(fields_autoplaced yes)
-		(property "Reference" "R740"
+		(property "Reference" "R540"
 			(at 35.56 71.1199 0)
 			(effects
@@
 			(project "y_board"
 				(path "/b3bc71fd-0ca0-4281-9bf5-aadd2561d695/b76c5e00-b7dd-4fa5-9261-12497b90aceb"
-					(reference "R740")
+					(reference "R540")
 					(unit 1)
 				)
@@
 		(dnp no)
 		(fields_autoplaced yes)
-		(property "Reference" "R743"
+		(property "Reference" "R543"
 			(at 67.31 71.1199 0)
 			(effects
@@
 			(project "y_board"
 				(path "/b3bc71fd-0ca0-4281-9bf5-aadd2561d695/b76c5e00-b7dd-4fa5-9261-12497b90aceb"
-					(reference "R743")
+					(reference "R543")
 					(unit 1)
 				)
@@
 					(unit 1)
 				)
-			)
-		)
-	)
-	(symbol
-		(lib_id "irf_s21850:S21850")
-		(at 68.58 120.65 0)
-		(unit 1)
-		(exclude_from_sim no)
-		(in_bom yes)
-		(on_board yes)
-		(dnp no)
-		(property "Reference" "IC703"
-			(at 68.58 119.38 0)
-			(effects
-				(font
-					(size 1.27 1.27)
-				)
-			)
-		)
-		(property "Value" "~"
-			(at 68.58 119.38 0)
-			(effects
-				(font
-					(size 1.27 1.27)
-				)
-			)
-		)
-		(property "Footprint" ""
-			(at 67.31 123.19 0)
-			(effects
-				(font
-					(size 1.27 1.27)
-				)
-				(hide yes)
-			)
-		)
-		(property "Datasheet" ""
-			(at 67.31 123.19 0)
-			(effects
-				(font
-					(size 1.27 1.27)
-				)
-				(hide yes)
-			)
-		)
-		(property "Description" ""
-			(at 67.31 123.19 0)
-			(effects
-				(font
-					(size 1.27 1.27)
-				)
-				(hide yes)
-			)
-		)
-		(pin "6"
-		)
-		(pin "8"
-		)
-		(pin "4"
-		)
-		(pin "3"
-		)
-		(pin "2"
-		)
-		(pin "1"
-		)
-		(pin "5"
-		)
-		(pin "7"
-		)
-		(instances
-			(project ""
-				(path "/b3bc71fd-0ca0-4281-9bf5-aadd2561d695/b76c5e00-b7dd-4fa5-9261-12497b90aceb"
-					(reference "IC703")
-					(unit 1)
-				)

Commit message: Modify optocouple "Unknown IC" after test
Parts:
- IC601: value ~ -> Unknown IC
Connections:
- no-connect marks 2 -> 5
Changed lines of the file:
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@@
 	)
 	(no_connect
+		(at 226.06 81.28)
+	)
+	(no_connect
 		(at 60.96 129.54)
 	)
+	(no_connect
+		(at 208.28 78.74)
+	)
+	(no_connect
+		(at 208.28 86.36)
+	)
 	(wire
 		(pts
@@
 	(wire
 		(pts
-			(xy 227.33 86.36) (xy 246.38 86.36)
+			(xy 226.06 86.36) (xy 246.38 86.36)
 		)
 		(stroke
@@
 	(wire
 		(pts
-			(xy 227.33 78.74) (xy 234.95 78.74)
+			(xy 226.06 78.74) (xy 234.95 78.74)
 		)
 		(stroke
@@
 	(wire
 		(pts
-			(xy 209.55 83.82) (xy 184.15 83.82)
+			(xy 208.28 83.82) (xy 184.15 83.82)
 		)
 		(stroke
@@
 	(wire
 		(pts
-			(xy 233.68 83.82) (xy 227.33 83.82)
+			(xy 233.68 83.82) (xy 226.06 83.82)
 		)
 		(stroke
@@
 	(wire
 		(pts
-			(xy 195.58 81.28) (xy 209.55 81.28)
+			(xy 195.58 81.28) (xy 208.28 81.28)
 		)
 		(stroke
@@
 	)
 	(symbol
-		(lib_id "irf_s21850:3411918")
-		(at 218.44 74.93 0)
-		(unit 1)
-		(exclude_from_sim no)
-		(in_bom yes)
-		(on_board yes)
-		(dnp no)
-		(property "Reference" "IC601"
-			(at 218.44 72.39 0)
-			(effects
-				(font
-					(size 1.27 1.27)
-				)
-			)
-		)
-		(property "Value" "~"
-			(at 218.44 73.66 0)
-			(effects
-				(font
-					(size 1.27 1.27)
-				)
-			)
-		)
-		(property "Footprint" ""
-			(at 218.44 74.93 0)
-			(effects
-				(font
-					(size 1.27 1.27)
-				)
-				(hide yes)
-			)
-		)
-		(property "Datasheet" ""
-			(at 218.44 74.93 0)
-			(effects
-				(font
-					(size 1.27 1.27)
-				)
-				(hide yes)
-			)
-		)
-		(property "Description" ""
-			(at 218.44 74.93 0)
-			(effects
-				(font
-					(size 1.27 1.27)
-				)
-				(hide yes)
-			)
-		)
-		(pin "8"
-		)
-		(pin "7"
-		)
-		(pin "4"
-		)
-		(pin "6"
-		)
-		(pin "1"
-		)
-		(pin "2"
-		)
-		(pin "3"
-		)
-		(pin "5"
-		)
-		(instances
-			(project ""
-				(path "/b3bc71fd-0ca0-4281-9bf5-aadd2561d695/b76c5e00-b7dd-4fa5-9261-12497b90aceb"
-					(reference "IC601")
-					(unit 1)
-				)
-			)
-		)
-	)
-	(symbol
 		(lib_id "power:Earth")
 		(at 33.02 87.63 0)
@@
 					(unit 1)
 				)
+			)
+		)
+	)
+	(symbol
+		(lib_name "3411918_1")
+		(lib_id "irf_s21850:3411918")
+		(at 217.17 74.93 0)
+		(unit 1)
+		(exclude_from_sim no)
+		(in_bom yes)
+		(on_board yes)
+		(dnp no)
+		(fields_autoplaced yes)
+		(property "Reference" "IC601"
+			(at 217.17 71.12 0)
+			(effects
+				(font
+					(size 1.27 1.27)
+				)
+			)
+		)
+		(property "Value" "Unknown IC"
+			(at 217.17 73.66 0)
+			(effects
+				(font
+					(size 1.27 1.27)
+				)
+			)
+		)
+		(property "Footprint" ""
+			(at 217.17 74.93 0)
+			(effects
+				(font
+					(size 1.27 1.27)
+				)
+				(hide yes)
+			)
+		)
+		(property "Datasheet" ""
+			(at 217.17 74.93 0)
+			(effects
+				(font
+					(size 1.27 1.27)
+				)
+				(hide yes)
+			)
+		)
+		(property "Description" ""
+			(at 217.17 74.93 0)
+			(effects
+				(font
+					(size 1.27 1.27)
+				)
+				(hide yes)
+			)
+		)
+		(pin "8"
+		)
+		(pin "7"
+		)
+		(pin "5"
+		)
+		(pin "3"
+		)
+		(pin "6"
+		)
+		(pin "4"
+		)
+		(pin "2"
+		)
+		(pin "1"
+		)
+		(instances
+			(project ""
+				(path "/b3bc71fd-0ca0-4281-9bf5-aadd2561d695/b76c5e00-b7dd-4fa5-9261-12497b90aceb"
+					(reference "IC601")
+					(unit 1)
+				)

Commit message: Update Y-Board schematics and add Y-Board top detailed information
Parts:
- C202: value ~ -> 330uF/25V
Changed lines of the file:
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@@
 		(on_board yes)
 		(dnp no)
-		(fields_autoplaced yes)
 		(property "Reference" "C202"
-			(at 91.44 85.9281 0)
+			(at 80.01 87.63 0)
 			(effects
 				(font
@@
 			)
 		)
-		(property "Value" "~"
-			(at 91.44 88.4681 0)
+		(property "Value" "330uF/25V"
+			(at 77.47 91.44 0)
 			(effects
 				(font

Commit message: Finishing document detailed images
Changed lines of the file:
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@@
 		(dnp no)
 		(property "Reference" "IC703"
-			(at 68.58 118.11 0)
+			(at 68.58 119.38 0)
 			(effects
 				(font
@@
 		)
 		(property "Value" "S21850"
-			(at 68.58 118.11 0)
+			(at 68.58 135.89 0)
 			(effects
 				(font
 					(size 1.27 1.27)
 				)
-				(hide yes)
 			)
 		)

Commit message: Update Power transistor names
Parts:
- D12: value D_Filled -> RF2001
- Q15: value NMOS -> IRFP4332
- Q16: value Q_NIGBT_GCE -> IRGP4086
Changed lines of the file:
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@@
 		(dnp no)
 		(property "Reference" "Q15"
-			(at 173.99 125.7299 0)
-			(effects
-				(font
-					(size 1.27 1.27)
-				)
-				(justify left)
-			)
-		)
-		(property "Value" "NMOS"
-			(at 173.99 128.2699 0)
-			(effects
-				(font
-					(size 1.27 1.27)
-				)
-				(justify left)
-				(hide yes)
+			(at 182.88 119.38 0)
+			(effects
+				(font
+					(size 1.27 1.27)
+				)
+				(justify left)
+			)
+		)
+		(property "Value" "IRFP4332"
+			(at 187.96 121.92 0)
+			(effects
+				(font
+					(size 1.27 1.27)
+				)
+				(justify left)
 			)
 		)
@@
 			)
 		)
-		(property "Value" "Q_NIGBT_GCE"
+		(property "Value" "IRGP4086"
 			(at 128.27 128.2699 0)
 			(effects
@@
 				)
 				(justify left)
-				(hide yes)
 			)
 		)
@@
 			)
 		)
-		(property "Value" "D_Filled"
+		(property "Value" "RF2001"
 			(at 146.05 128.2699 90)
 			(effects
@@
 				)
 				(justify left)
-				(hide yes)
-			)
-		)
+			)
+		)
