File: TV_PLASMA/42PQ30R/y_board/y_board.kicad_sch (KiCad schematic)
At the start: 7 parts

Commit message: Add Set Up circuit to schematic
Other:
- added sheet SetUp (set_up.kicad_sch)
Changed lines of the file:
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@@
+	)
+	(sheet
+		(at -34.29 113.03)
+		(size 22.86 17.78)
+		(fields_autoplaced yes)
+		(stroke
+			(width 0.1524)
+			(type solid)
+		)
+		(fill
+			(color 0 0 0 0.0000)
+		)
+		(property "Sheetname" "SetUp"
+			(at -34.29 112.3184 0)
+			(effects
+				(font
+					(size 1.27 1.27)
+				)
+				(justify left bottom)
+			)
+		)
+		(property "Sheetfile" "set_up.kicad_sch"
+			(at -34.29 131.3946 0)
+			(effects
+				(font
+					(size 1.27 1.27)
+				)
+				(justify left top)
+			)
+		)
+		(instances
+			(project "y_board"
+				(path "/b3bc71fd-0ca0-4281-9bf5-aadd2561d695"
+					(page "5")
+				)
+			)
+		)
 	)
 	(sheet
@@
 	(sheet
 		(at -39.37 73.66)
-		(size 27.94 27.94)
+		(size 24.13 21.59)
 		(fields_autoplaced yes)
 		(stroke
@@
 		)
 		(property "Sheetfile" "y_er_up_and_sus_up.kicad_sch"
-			(at -39.37 102.1846 0)
+			(at -39.37 95.8346 0)
 			(effects
 				(font

Commit message: Add Set Down circuit
Other:
- sheet Y_SUS_UP_AND_Y_BLOCKING renamed Y_SUS_DOWN_AND_Y_BLOCKING
- added sheet SetDown (set_down.kicad_sch)
Changed lines of the file:
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@@
 	)
 	(sheet
-		(at -34.29 113.03)
+		(at -39.37 128.27)
+		(size 21.59 17.78)
+		(fields_autoplaced yes)
+		(stroke
+			(width 0.1524)
+			(type solid)
+		)
+		(fill
+			(color 0 0 0 0.0000)
+		)
+		(property "Sheetname" "SetDown"
+			(at -39.37 127.5584 0)
+			(effects
+				(font
+					(size 1.27 1.27)
+				)
+				(justify left bottom)
+			)
+		)
+		(property "Sheetfile" "set_down.kicad_sch"
+			(at -39.37 146.6346 0)
+			(effects
+				(font
+					(size 1.27 1.27)
+				)
+				(justify left top)
+			)
+		)
+		(instances
+			(project "y_board"
+				(path "/b3bc71fd-0ca0-4281-9bf5-aadd2561d695"
+					(page "6")
+				)
+			)
+		)
+	)
+	(sheet
+		(at -39.37 102.87)
 		(size 22.86 17.78)
 		(fields_autoplaced yes)
@@
 		)
 		(property "Sheetname" "SetUp"
-			(at -34.29 112.3184 0)
+			(at -39.37 102.1584 0)
 			(effects
 				(font
@@
 		)
 		(property "Sheetfile" "set_up.kicad_sch"
-			(at -34.29 131.3946 0)
+			(at -39.37 121.2346 0)
 			(effects
 				(font
@@
 			(color 0 0 0 0.0000)
 		)
-		(property "Sheetname" "Y_SUS_UP_AND_Y_BLOCKING"
+		(property "Sheetname" "Y_SUS_DOWN_AND_Y_BLOCKING"
 			(at -39.37 18.3384 0)
 			(effects
