File: TV_PLASMA/42PQ30R/y_board/y_board.kicad_sch (KiCad schematic)
At the start: 7 parts

Commit message: Begin VY and VSC circuit (Part 2 of 3)
Other:
- added sheet VSC AND VY (Part 1 of 3) (vsc_and_vy.kicad_sch)
- added sheet VSC and VY (Part 2 of 3) (vcs_and_vy_part2_of_3.kicad_sch)
Changed lines of the file:
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@@
+	)
+	(sheet
+		(at -34.29 186.69)
+		(size 16.51 12.7)
+		(fields_autoplaced yes)
+		(stroke
+			(width 0.1524)
+			(type solid)
+		)
+		(fill
+			(color 0 0 0 0.0000)
+		)
+		(property "Sheetname" "VSC and VY (Part 2 of 3)"
+			(at -34.29 185.9784 0)
+			(effects
+				(font
+					(size 1.27 1.27)
+				)
+				(justify left bottom)
+			)
+		)
+		(property "Sheetfile" "vcs_and_vy_part2_of_3.kicad_sch"
+			(at -34.29 199.9746 0)
+			(effects
+				(font
+					(size 1.27 1.27)
+				)
+				(justify left top)
+			)
+		)
+		(instances
+			(project "y_board"
+				(path "/b3bc71fd-0ca0-4281-9bf5-aadd2561d695"
+					(page "8")
+				)
+			)
+		)
+	)
+	(sheet
+		(at -36.83 156.21)
+		(size 20.32 16.51)
+		(fields_autoplaced yes)
+		(stroke
+			(width 0.1524)
+			(type solid)
+		)
+		(fill
+			(color 0 0 0 0.0000)
+		)
+		(property "Sheetname" "VSC AND VY (Part 1 of 3)"
+			(at -36.83 155.4984 0)
+			(effects
+				(font
+					(size 1.27 1.27)
+				)
+				(justify left bottom)
+			)
+		)
+		(property "Sheetfile" "vsc_and_vy.kicad_sch"
+			(at -36.83 173.3046 0)
+			(effects
+				(font
+					(size 1.27 1.27)
+				)
+				(justify left top)
+			)
+		)
+		(instances
+			(project "y_board"
+				(path "/b3bc71fd-0ca0-4281-9bf5-aadd2561d695"
+					(page "7")
+				)
+			)
+		)
 	)
 	(sheet

Commit message: Finishing VSC and VY supply
Other:
- added sheet VSC and VY (Part 3 of 3) (vsc_and_vy_part3_of_3.kicad_sch)
Changed lines of the file:
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@@
 	)
 	(sheet
-		(at -39.37 128.27)
-		(size 21.59 17.78)
+		(at -38.1 92.71)
+		(size 20.32 10.16)
 		(fields_autoplaced yes)
 		(stroke
@@
 		)
 		(property "Sheetname" "SetDown"
-			(at -39.37 127.5584 0)
+			(at -38.1 91.9984 0)
 			(effects
 				(font
@@
 		)
 		(property "Sheetfile" "set_down.kicad_sch"
-			(at -39.37 146.6346 0)
+			(at -38.1 103.4546 0)
 			(effects
 				(font
@@
 	)
 	(sheet
-		(at -34.29 186.69)
-		(size 16.51 12.7)
+		(at -35.56 134.62)
+		(size 16.51 8.89)
 		(fields_autoplaced yes)
 		(stroke
@@
 		)
 		(property "Sheetname" "VSC and VY (Part 2 of 3)"
-			(at -34.29 185.9784 0)
+			(at -35.56 133.9084 0)
 			(effects
 				(font
@@
 		)
 		(property "Sheetfile" "vcs_and_vy_part2_of_3.kicad_sch"
-			(at -34.29 199.9746 0)
+			(at -35.56 144.0946 0)
 			(effects
 				(font
@@
 	)
 	(sheet
-		(at -36.83 156.21)
-		(size 20.32 16.51)
+		(at -36.83 113.03)
+		(size 20.32 11.43)
 		(fields_autoplaced yes)
 		(stroke
@@
 		)
 		(property "Sheetname" "VSC AND VY (Part 1 of 3)"
-			(at -36.83 155.4984 0)
+			(at -36.83 112.3184 0)
 			(effects
 				(font
@@
 		)
 		(property "Sheetfile" "vsc_and_vy.kicad_sch"
-			(at -36.83 173.3046 0)
+			(at -36.83 125.0446 0)
 			(effects
 				(font
@@
 	)
 	(sheet
-		(at -39.37 102.87)
-		(size 22.86 17.78)
+		(at -38.1 73.66)
+		(size 19.05 11.43)
 		(fields_autoplaced yes)
 		(stroke
@@
 		)
 		(property "Sheetname" "SetUp"
-			(at -39.37 102.1584 0)
+			(at -38.1 72.9484 0)
 			(effects
 				(font
@@
 		)
 		(property "Sheetfile" "set_up.kicad_sch"
-			(at -39.37 121.2346 0)
+			(at -38.1 85.6746 0)
 			(effects
 				(font
@@
 	)
 	(sheet
-		(at -39.37 44.45)
-		(size 25.4 20.32)
+		(at -39.37 35.56)
+		(size 17.78 11.43)
 		(fields_autoplaced yes)
 		(stroke
@@
 		)
 		(property "Sheetname" "y_er_down"
-			(at -39.37 43.7384 0)
+			(at -39.37 34.8484 0)
 			(effects
 				(font
@@
 		)
 		(property "Sheetfile" "y_er_down.kicad_sch"
-			(at -39.37 65.3546 0)
+			(at -39.37 47.5746 0)
 			(effects
 				(font
@@
 	(sheet
 		(at -39.37 19.05)
-		(size 21.59 16.51)
+		(size 19.05 10.16)
 		(fields_autoplaced yes)
 		(stroke
@@
 		)
 		(property "Sheetfile" "y_sus_dn_and_blocking.kicad_sch"
-			(at -39.37 36.1446 0)
+			(at -39.37 29.7946 0)
 			(effects
 				(font
@@
 	)
 	(sheet
-		(at -39.37 73.66)
-		(size 24.13 21.59)
+		(at -39.37 55.88)
+		(size 20.32 10.16)
 		(fields_autoplaced yes)
 		(stroke
@@
 		)
 		(property "Sheetname" "y_er_up_and_sus_up"
-			(at -39.37 72.9484 0)
+			(at -39.37 55.1684 0)
 			(effects
 				(font
@@
 		)
 		(property "Sheetfile" "y_er_up_and_sus_up.kicad_sch"
-			(at -39.37 95.8346 0)
+			(at -39.37 66.6246 0)
 			(effects
 				(font
@@
 				)
 			)
+		)
+	)
+	(sheet
+		(at -33.02 153.67)
+		(size 12.7 10.16)
+		(fields_autoplaced yes)
+		(stroke
+			(width 0.1524)
+			(type solid)
+		)
+		(fill
+			(color 0 0 0 0.0000)
+		)
+		(property "Sheetname" "VSC and VY (Part 3 of 3)"
+			(at -33.02 152.9584 0)
+			(effects
+				(font
+					(size 1.27 1.27)
+				)
+				(justify left bottom)
+			)
+		)
+		(property "Sheetfile" "vsc_and_vy_part3_of_3.kicad_sch"
+			(at -33.02 164.4146 0)
+			(effects
+				(font
+					(size 1.27 1.27)
+				)
+				(justify left top)
+			)
+		)
+		(instances
+			(project "y_board"
+				(path "/b3bc71fd-0ca0-4281-9bf5-aadd2561d695"
+					(page "9")
+				)
+			)

Commit message: Ordering page priotity and removing TODO
Parts:
- added C203: 330uF/25V, symbol Device:C_Polarized_Small_US
- added C221: 150uF/150V, symbol Device:C_Polarized_Small_US
- added P201: Conn_01x10_Pin, symbol Connector:Conn_01x10_Pin
- added P202: Conn_01x07_Pin, symbol Connector:Conn_01x07_Pin
- C205, C206, C207, C208: value C_Polarized_Small_US -> 220uF/250V
Connections:
- net Earth: now also C203.2, C221.2, P201.4 (Pin_4), P201.5 (Pin_5), P201.8 (Pin_8), P202.1 (Pin_1), P202.2 (Pin_2), P202.3 (Pin_3)
- net at FL201.1: now also P201.1 (Pin_1), P201.2 (Pin_2)
- new net 5V: C203.1, P201.10 (Pin_10), P201.9 (Pin_9)
- new net VA: C221.1, P201.6 (Pin_6), P201.7 (Pin_7), P202.5 (Pin_5), P202.6 (Pin_6), P202.7 (Pin_7)
- no-connect marks 0 -> 2
Other:
- note added: "P201 (Input Power Supply) 1- +VS 2- +VS 3- NC 4- GND 5- GND 6- +VA 7- +VA 8- GND 9- +5V 10- +5V"
- note added: "P202 (Output VA Supply) 1- GND 2- GND 3- GND 4- NC 5- +VA 6- +VA 7- +VA"
- note removed: "TODO: - Add voltage pins - Add capacitor values"
- moved on the sheet: C205, C206, C207, C208, C209, FL201, FS201

Commit message: Finishing 15VF, 5VF and 15V power supply
Other:
- added sheet 5VF, 15VF 15v (5VF_15VF_15V.kicad_sch)
Changed lines of the file:
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@@
 			(project "y_board"
 				(path "/b3bc71fd-0ca0-4281-9bf5-aadd2561d695"
-					(page "9")
+					(page "10")
 				)
 			)
@@
 			(project "y_board"
 				(path "/b3bc71fd-0ca0-4281-9bf5-aadd2561d695"
-					(page "3")
+					(page "4")
 				)
 			)
@@
 			(project "y_board"
 				(path "/b3bc71fd-0ca0-4281-9bf5-aadd2561d695"
-					(page "2")
+					(page "3")
 				)
 			)
@@
 			(project "y_board"
 				(path "/b3bc71fd-0ca0-4281-9bf5-aadd2561d695"
-					(page "8")
+					(page "9")
+				)
+			)
+		)
+	)
+	(sheet
+		(at -31.75 173.99)
+		(size 16.51 12.7)
+		(fields_autoplaced yes)
+		(stroke
+			(width 0.1524)
+			(type solid)
+		)
+		(fill
+			(color 0 0 0 0.0000)
+		)
+		(property "Sheetname" "5VF, 15VF 15v"
+			(at -31.75 173.2784 0)
+			(effects
+				(font
+					(size 1.27 1.27)
+				)
+				(justify left bottom)
+			)
+		)
+		(property "Sheetfile" "5VF_15VF_15V.kicad_sch"
+			(at -31.75 187.2746 0)
+			(effects
+				(font
+					(size 1.27 1.27)
+				)
+				(justify left top)
+			)
+		)
+		(instances
+			(project "y_board"
+				(path "/b3bc71fd-0ca0-4281-9bf5-aadd2561d695"
+					(page "2")
 				)
 			)
@@
 			(project "y_board"
 				(path "/b3bc71fd-0ca0-4281-9bf5-aadd2561d695"
-					(page "6")
+					(page "7")
 				)
 			)
@@
 			(project "y_board"
 				(path "/b3bc71fd-0ca0-4281-9bf5-aadd2561d695"
-					(page "5")
+					(page "6")
 				)
 			)
@@
 			(project "y_board"
 				(path "/b3bc71fd-0ca0-4281-9bf5-aadd2561d695"
-					(page "7")
+					(page "8")
 				)
 			)
@@
 			(project "y_board"
 				(path "/b3bc71fd-0ca0-4281-9bf5-aadd2561d695"
-					(page "4")
-				)
-			)
+					(page "5")
+				)
+			)

Commit message: Add control input parts 2,3 of 3
Other:
- added sheet Input control (Part 1 of 3) (input_control.kicad_sch)
- added sheet Input control (Part 2 of 3) (input_control2.kicad_sch)
- added sheet Input control (Part 3 of 3) (input_control3.kicad_sch)
- moved on the sheet: C203, C205, C206, C207, C208, C209, C221, FL201, FS201, P201, P202

Commit message: Implement Output Control
Other:
- added sheet Output Control (Part 1 of 3) (output_control.kicad_sch)
- added sheet Output Control (Part 2 of 3) (output_control2.kicad_sch)
Changed lines of the file:
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@@
+	)
+	(sheet
+		(at 311.15 55.88)
+		(size 17.78 13.97)
+		(fields_autoplaced yes)
+		(stroke
+			(width 0.1524)
+			(type solid)
+		)
+		(fill
+			(color 0 0 0 0.0000)
+		)
+		(property "Sheetname" "Output Control (Part 1 of 3)"
+			(at 311.15 55.1684 0)
+			(effects
+				(font
+					(size 1.27 1.27)
+				)
+				(justify left bottom)
+			)
+		)
+		(property "Sheetfile" "output_control.kicad_sch"
+			(at 311.15 70.4346 0)
+			(effects
+				(font
+					(size 1.27 1.27)
+				)
+				(justify left top)
+			)
+		)
+		(instances
+			(project "y_board"
+				(path "/b3bc71fd-0ca0-4281-9bf5-aadd2561d695"
+					(page "14")
+				)
+			)
+		)
 	)
 	(sheet
@@
 				)
 			)
+		)
+	)
+	(sheet
+		(at 313.69 91.44)
+		(size 12.7 11.43)
+		(fields_autoplaced yes)
+		(stroke
+			(width 0.1524)
+			(type solid)
+		)
+		(fill
+			(color 0 0 0 0.0000)
+		)
+		(property "Sheetname" "Output Control (Part 2 of 3)"
+			(at 313.69 90.7284 0)
+			(effects
+				(font
+					(size 1.27 1.27)
+				)
+				(justify left bottom)
+			)
+		)
+		(property "Sheetfile" "output_control2.kicad_sch"
+			(at 313.69 103.4546 0)
+			(effects
+				(font
+					(size 1.27 1.27)
+				)
+				(justify left top)
+			)
+		)
+		(instances
+			(project "y_board"
+				(path "/b3bc71fd-0ca0-4281-9bf5-aadd2561d695"
+					(page "15")
+				)
+			)

Commit message: Finishing Y BOARD reverse engineering. Todo: Add reverse conduction and resistence to all output/input pins and refactor Z BOARD DRC
Other:
- sheet Output Control (Part 1 of 3) renamed Output Control (Part 1 of 4)
- sheet Output Control (Part 2 of 3) renamed Output Control (Part 2 of 4)
- added sheet Output Control (Part 3 of 4) (output_control3.kicad_sch)
- added sheet Output Control (Part 4 of 4) (output_control4.kicad_sch)
- note added: "VOLTAGES SUPPLY"
Changed lines of the file:
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@@
-	)
-	(junction
-		(at 139.7 67.31)
-		(diameter 0)
-		(color 0 0 0 0)
 	)
 	(junction
@@
 	)
 	(junction
+		(at 151.13 67.31)
+		(diameter 0)
+		(color 0 0 0 0)
+	)
+	(junction
 		(at 214.63 82.55)
 		(diameter 0)
@@
 	(wire
 		(pts
+			(xy 151.13 67.31) (xy 151.13 74.93)
+		)
+		(stroke
+			(width 0)
+			(type default)
+		)
+	)
+	(wire
+		(pts
 			(xy 101.6 57.15) (xy 105.41 57.15)
 		)
@@
 	(wire
 		(pts
-			(xy 154.94 67.31) (xy 139.7 67.31)
-		)
-		(stroke
-			(width 0)
-			(type default)
-		)
-	)
-	(wire
-		(pts
 			(xy 119.38 54.61) (xy 127 54.61)
 		)
@@
 	(wire
 		(pts
-			(xy 139.7 67.31) (xy 139.7 69.85)
-		)
-		(stroke
-			(width 0)
-			(type default)
-		)
-	)
-	(wire
-		(pts
 			(xy 104.14 77.47) (xy 104.14 74.93)
 		)
@@
 	(wire
 		(pts
+			(xy 139.7 67.31) (xy 151.13 67.31)
+		)
+		(stroke
+			(width 0)
+			(type default)
+		)
+	)
+	(wire
+		(pts
 			(xy 214.63 82.55) (xy 218.44 82.55)
 		)
@@
 			(width 0)
 			(type default)
+		)
+	)
+	(wire
+		(pts
+			(xy 151.13 67.31) (xy 154.94 67.31)
+		)
+		(stroke
+			(width 0)
+			(type default)
+		)
+	)
+	(text "VOLTAGES SUPPLY"
+		(exclude_from_sim no)
+		(at 151.13 21.59 0)
+		(effects
+			(font
+				(size 5 5)
+				(thickness 0.6)
+				(bold yes)
+				(italic yes)
+			)
 		)
 	)
@@
 			)
 			(justify left)
-		)
-	)
-	(label "VOLTAGES SUPPLY"
-		(at 177.8 25.4 180)
-		(effects
-			(font
-				(face "KiCad Font")
-				(size 5 5)
-				(thickness 0.254)
-				(bold yes)
-				(italic yes)
-			)
-			(justify right bottom)
 		)
 	)
@@
 	(symbol
 		(lib_id "power:Earth")
-		(at 139.7 69.85 0)
+		(at 151.13 74.93 0)
 		(unit 1)
 		(exclude_from_sim no)
@@
 		(fields_autoplaced yes)
 		(property "Reference" "#PWR1"
-			(at 139.7 76.2 0)
+			(at 151.13 81.28 0)
 			(effects
 				(font
@@
 		)
 		(property "Value" "Earth"
-			(at 139.7 74.93 0)
+			(at 151.13 80.01 0)
 			(effects
 				(font
@@
 		)
 		(property "Footprint" ""
-			(at 139.7 69.85 0)
+			(at 151.13 74.93 0)
 			(effects
 				(font
@@
 		)
 		(property "Datasheet" "~"
-			(at 139.7 69.85 0)
+			(at 151.13 74.93 0)
 			(effects
 				(font
@@
 		)
 		(property "Description" "Power symbol creates a global label with name \"Earth\""
-			(at 139.7 69.85 0)
+			(at 151.13 74.93 0)
 			(effects
 				(font
@@
 	)
 	(sheet
+		(at 309.88 137.16)
+		(size 16.51 11.43)
+		(fields_autoplaced yes)
+		(stroke
+			(width 0.1524)
+			(type solid)
+		)
+		(fill
+			(color 0 0 0 0.0000)
+		)
+		(property "Sheetname" "Output Control (Part 4 of 4)"
+			(at 309.88 136.4484 0)
+			(effects
+				(font
+					(size 1.27 1.27)
+				)
+				(justify left bottom)
+			)
+		)
+		(property "Sheetfile" "output_control4.kicad_sch"
+			(at 309.88 149.1746 0)
+			(effects
+				(font
+					(size 1.27 1.27)
+				)
+				(justify left top)
+			)
+		)
+		(instances
+			(project "y_board"
+				(path "/b3bc71fd-0ca0-4281-9bf5-aadd2561d695"
+					(page "17")
+				)
+			)
+		)
+	)
+	(sheet
 		(at -33.02 196.85)
 		(size 20.32 10.16)
@@
 			(color 0 0 0 0.0000)
 		)
-		(property "Sheetname" "Output Control (Part 1 of 3)"
+		(property "Sheetname" "Output Control (Part 1 of 4)"
 			(at 311.15 55.1684 0)
 			(effects
@@
 	)
 	(sheet
+		(at 311.15 115.57)
+		(size 13.97 10.16)
+		(fields_autoplaced yes)
+		(stroke
+			(width 0.1524)
+			(type solid)
+		)
+		(fill
+			(color 0 0 0 0.0000)
+		)
+		(property "Sheetname" "Output Control (Part 3 of 4)"
+			(at 311.15 114.8584 0)
+			(effects
+				(font
+					(size 1.27 1.27)
+				)
+				(justify left bottom)
+			)
+		)
+		(property "Sheetfile" "output_control3.kicad_sch"
+			(at 311.15 126.3146 0)
+			(effects
+				(font
+					(size 1.27 1.27)
+				)
+				(justify left top)
+			)
+		)
+		(instances
+			(project "y_board"
+				(path "/b3bc71fd-0ca0-4281-9bf5-aadd2561d695"
+					(page "16")
+				)
+			)
+		)
+	)
+	(sheet
 		(at -39.37 35.56)
 		(size 17.78 11.43)
@@
 			(color 0 0 0 0.0000)
 		)
-		(property "Sheetname" "Output Control (Part 2 of 3)"
+		(property "Sheetname" "Output Control (Part 2 of 4)"
 			(at 313.69 90.7284 0)
 			(effects

Commit message: Finishing reverse engineering Y BOARD
Other:
- added sheet Measurements P101 (measurements_p101.kicad_sch)
- added sheet Measurements P201 (measurements.kicad_sch)
- added sheet Measurements P202 (measurements_p202.kicad_sch)
- added sheet Measurements P203, P208 and P205 (measurements_p203_p208_p205.kicad_sch)
- added sheet Measurements P206 (measurements_p206.kicad_sch)
- added sheet Measurements P207 (measurements_p207.kicad_sch)
- moved on the sheet: C203, C205, C206, C207, C208, C209, C221, FL201, FS201, P201, P202
