File: TV_PLASMA/42PQ30R/y_board/y_board.kicad_sch (KiCad schematic)
At the start: 11 parts, among them P201 Conn_01x10_Pin, P202 Conn_01x07_Pin

Commit message: Update Y-Board schematics and add Y-Board top detailed information
Parts:
- C209: value C -> 3.3uF/250V
Changed lines of the file:
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@@
 			)
 		)
-		(property "Value" "C"
+		(property "Value" "3.3uF/250V"
 			(at 195.58 73.6599 0)
 			(effects
@@
 				)
 				(justify left)
-				(hide yes)
 			)
 		)
