File: TV_PLASMA/42PQ30R/y_board/input_control.kicad_sch (KiCad schematic)
At the start: 0 parts

Commit message: Finishing implementing output control
Parts:
- added P101: Conn_02x15_Counter_Clockwise, symbol Connector_Generic:Conn_02x15_Counter_Clockwise
Connections:
- new net 15V: P101.1 (Pin_1), P101.30 (Pin_30)
- new net 5V: P101.2 (Pin_2), P101.28 (Pin_28), P101.29 (Pin_29), P101.3 (Pin_3), P101.4 (Pin_4)
- new net CTRL_OE: P101.17 (Pin_17)
- new net Earth: P101.16 (Pin_16), P101.26 (Pin_26), P101.27 (Pin_27), P101.5 (Pin_5), P101.6 (Pin_6)
- new net I_CLK: P101.20 (Pin_20)
- new net I_DATA: P101.23 (Pin_23)
- new net I_DELTA_VY_DET: P101.25 (Pin_25)
- new net I_DET_LEVEL_SEL: P101.19 (Pin_19)
- new net I_OC1: P101.22 (Pin_22)
- new net I_OC2: P101.24 (Pin_24)
- new net I_PASS_TOP: P101.12 (Pin_12)
- new net I_RAMP_SLOPE_OPT: P101.11 (Pin_11)
- new net I_SET_DN: P101.15 (Pin_15)
- new net I_SET_UP: P101.10 (Pin_10)
- new net I_SLOPE_RATE_SEL: P101.18 (Pin_18)
- new net I_STB: P101.21 (Pin_21)
- new net I_SUS_DN_IN: P101.8 (Pin_8)
- new net I_SUS_UP_IN: P101.14 (Pin_14)
- new net I_YER_DN: P101.9 (Pin_9)
- new net I_YER_UP: P101.13 (Pin_13)
- new net OE: P101.7 (Pin_7)

Commit message: Finishing Y BOARD reverse engineering. Todo: Add reverse conduction and resistence to all output/input pins and refactor Z BOARD DRC
Other:
- note added: "30- 15V 29- 5V 28- 5V 27- GND 26- GND 25- (1 - I_DELTA_VY_DET) 24- (3- I_OC2) 23- (5- I_DATA) 22- (7- I_OC1) 21- (9- I_STB) 20- (11- I_CLK) 19- (13- I_DET_LEVEL_SEL) 18- (15- I_SLOPE_RATE_SEL) 17- (17- I_CTRL_OE) 16- GND"
- note added: "Input Control (Part 1 of 3)"
- note added: "P101 1- 15V 2- 5V 3- 5V 4- 5V 5- GND 6- GND 7- (2- OE) 8- (4- I_YSUS_DN_IN) 9- (6- I_YER_DN) 10- (8- I_SET_UP) 11- (10- I_RAMP_SLOPE_OPT) 12- (12- I_PASS_TOP) 13- (14- I_YER_UP) 14- (16- I_SUS_UP_IN) 15- (18- I_SET_DN)"
- moved on the sheet: P101

Commit message: Finishing reverse engineering Y BOARD
Changed lines of the file:
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@@
 	)
 	(global_label "OE"
-		(shape passive)
+		(shape input)
 		(at 92.71 101.6 180)
 		(fields_autoplaced yes)
@@
 		)
 		(property "Intersheetrefs" "${INTERSHEET_REFS}"
-			(at 88.3566 101.6 0)
+			(at 87.2453 101.6 0)
 			(effects
 				(font
