File: TV_PLASMA/42PQ30R/y_board/output_control4.kicad_sch (KiCad schematic)
At the start: 4 parts, among them P203 Conn_01x12_Pin, P205 Conn_01x12_Pin, P207 Conn_01x12_Pin, P208 Conn_01x12_Pin

Commit message: Finishing reverse engineering Y BOARD
Parts:
- added P206: Conn_01x08_Pin, symbol Connector:Conn_01x08_Pin
Connections:
- new net ER_CON: P206.1 (Pin_1), P206.2 (Pin_2)
- new net Earth: P206.4 (Pin_4), P206.5 (Pin_5)
- new net VS_B: P206.7 (Pin_7), P206.8 (Pin_8)
- no-connect marks 1 -> 3
Other:
- note added: "P206 1- ER_CON 2- ER_CON 3- NC 4- GND 5- GND 6- NC 7- +VS 8- +VS"
