File: TV_PLASMA/42PQ30R/y_board/vsc_and_vy_part3_of_3.kicad_sch (KiCad schematic)
At the start: 31 parts, among them IC303 EL817, Q302 Q_NPN_BCE, Q304 NMOS, Q304 Q_SCR_KGA

Commit message: Finishing 15VF, 5VF and 15V power supply
Connections:
- net 15VY is gone; now on net 15V: R324.1
Changed lines of the file:
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@@
 		)
 	)
-	(global_label "15VY"
+	(global_label "15V"
 		(shape input)
 		(at 58.42 43.18 180)
@@
 		)
 		(property "Intersheetrefs" "${INTERSHEET_REFS}"
-			(at 50.8386 43.18 0)
+			(at 51.9272 43.18 0)
 			(effects
 				(font

Commit message: Update Set Down Q information. Add label to VSC and VY supply
Parts:
- added R333: 1k, symbol Device:R
- renumbered Q304 to Q305
Connections:
- net 5V: now also R333.1
- net OE_IC102: now also R333.2
- net I_DET_LEVEL_SEL_A: now reaches C304.2, IC401.2 (IN1-), R309.2, R311.1, R320.1, ZD302.1 (K)
Other:
- moved on the sheet: R324
Changed lines of the file:
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@@
+	)
+	(junction
+		(at 109.22 38.1)
+		(diameter 0)
+		(color 0 0 0 0)
 	)
 	(junction
@@
 	)
 	(junction
+		(at 109.22 26.67)
+		(diameter 0)
+		(color 0 0 0 0)
+	)
+	(junction
 		(at 143.51 129.54)
 		(diameter 0)
@@
 	(wire
 		(pts
+			(xy 109.22 38.1) (xy 152.4 38.1)
+		)
+		(stroke
+			(width 0)
+			(type default)
+		)
+	)
+	(wire
+		(pts
 			(xy 209.55 157.48) (xy 217.17 157.48)
 		)
@@
 	(wire
 		(pts
-			(xy 55.88 36.83) (xy 137.16 36.83)
+			(xy 57.15 26.67) (xy 109.22 26.67)
 		)
 		(stroke
@@
 	(wire
 		(pts
-			(xy 167.64 154.94) (xy 167.64 144.78)
+			(xy 167.64 160.02) (xy 167.64 144.78)
 		)
 		(stroke
@@
 	(wire
 		(pts
+			(xy 100.33 151.13) (xy 158.75 151.13)
+		)
+		(stroke
+			(width 0)
+			(type default)
+		)
+	)
+	(wire
+		(pts
 			(xy 226.06 115.57) (xy 215.9 115.57)
 		)
@@
 	(wire
 		(pts
-			(xy 96.52 54.61) (xy 96.52 59.69)
+			(xy 96.52 57.15) (xy 96.52 59.69)
 		)
 		(stroke
@@
 	(wire
 		(pts
-			(xy 90.17 154.94) (xy 167.64 154.94)
+			(xy 90.17 160.02) (xy 167.64 160.02)
 		)
 		(stroke
@@
 	(wire
 		(pts
-			(xy 137.16 36.83) (xy 137.16 73.66)
-		)
-		(stroke
-			(width 0)
-			(type default)
-		)
-	)
-	(wire
-		(pts
-			(xy 58.42 43.18) (xy 96.52 43.18)
+			(xy 137.16 26.67) (xy 137.16 73.66)
+		)
+		(stroke
+			(width 0)
+			(type default)
+		)
+	)
+	(wire
+		(pts
+			(xy 58.42 45.72) (xy 96.52 45.72)
 		)
 		(stroke
@@
 	(wire
 		(pts
-			(xy 96.52 43.18) (xy 96.52 46.99)
+			(xy 96.52 45.72) (xy 96.52 49.53)
 		)
 		(stroke
@@
 	(wire
 		(pts
+			(xy 109.22 35.56) (xy 109.22 38.1)
+		)
+		(stroke
+			(width 0)
+			(type default)
+		)
+	)
+	(wire
+		(pts
 			(xy 215.9 115.57) (xy 215.9 129.54)
 		)
@@
 	(wire
 		(pts
-			(xy 152.4 30.48) (xy 152.4 85.09)
+			(xy 152.4 38.1) (xy 152.4 85.09)
 		)
 		(stroke
@@
 	(wire
 		(pts
-			(xy 60.96 30.48) (xy 152.4 30.48)
+			(xy 109.22 26.67) (xy 109.22 27.94)
+		)
+		(stroke
+			(width 0)
+			(type default)
+		)
+	)
+	(wire
+		(pts
+			(xy 62.23 38.1) (xy 109.22 38.1)
 		)
 		(stroke
@@
 	(wire
 		(pts
+			(xy 158.75 151.13) (xy 158.75 129.54)
+		)
+		(stroke
+			(width 0)
+			(type default)
+		)
+	)
+	(wire
+		(pts
 			(xy 120.65 111.76) (xy 120.65 115.57)
 		)
@@
 		(pts
 			(xy 181.61 144.78) (xy 187.96 144.78)
+		)
+		(stroke
+			(width 0)
+			(type default)
+		)
+	)
+	(wire
+		(pts
+			(xy 109.22 26.67) (xy 137.16 26.67)
 		)
 		(stroke
@@
 		)
 	)
-	(global_label "OE_IC102"
+	(global_label "I_DET_LEVEL_SEL_A"
 		(shape passive)
-		(at 60.96 30.48 180)
+		(at 100.33 151.13 180)
 		(fields_autoplaced yes)
 		(effects
@@
 		)
 		(property "Intersheetrefs" "${INTERSHEET_REFS}"
-			(at 50.1357 30.48 0)
+			(at 80.6763 151.13 0)
 			(effects
 				(font
@@
 		)
 	)
-	(global_label "VS_B"
-		(shape input)
-		(at 90.17 154.94 180)
+	(global_label "OE_IC102"
+		(shape passive)
+		(at 62.23 38.1 180)
 		(fields_autoplaced yes)
 		(effects
@@
 		)
 		(property "Intersheetrefs" "${INTERSHEET_REFS}"
-			(at 82.6491 154.94 0)
+			(at 51.4057 38.1 0)
 			(effects
 				(font
@@
 		)
 	)
-	(global_label "15V"
+	(global_label "VS_B"
 		(shape input)
-		(at 58.42 43.18 180)
+		(at 90.17 160.02 180)
 		(fields_autoplaced yes)
 		(effects
@@
 		)
 		(property "Intersheetrefs" "${INTERSHEET_REFS}"
-			(at 51.9272 43.18 0)
+			(at 82.6491 160.02 0)
+			(effects
+				(font
+					(size 1.27 1.27)
+				)
+				(justify right)
+				(hide yes)
+			)
+		)
+	)
+	(global_label "15V"
+		(shape input)
+		(at 58.42 45.72 180)
+		(fields_autoplaced yes)
+		(effects
+			(font
+				(size 1.27 1.27)
+			)
+			(justify right)
+		)
+		(property "Intersheetrefs" "${INTERSHEET_REFS}"
+			(at 51.9272 45.72 0)
 			(effects
 				(font
@@
 	(global_label "5V"
 		(shape input)
-		(at 55.88 36.83 180)
+		(at 57.15 26.67 180)
 		(fields_autoplaced yes)
 		(effects
@@
 		)
 		(property "Intersheetrefs" "${INTERSHEET_REFS}"
-			(at 50.5967 36.83 0)
+			(at 51.8667 26.67 0)
 			(effects
 				(font
@@
 	(symbol
 		(lib_id "Device:R")
-		(at 96.52 50.8 0)
+		(at 96.52 53.34 0)
 		(unit 1)
 		(exclude_from_sim no)
@@
 		(dnp no)
 		(property "Reference" "R324"
-			(at 97.79 49.53 0)
+			(at 97.79 52.07 0)
 			(effects
 				(font
@@
 		)
 		(property "Value" "1k"
-			(at 97.79 52.07 0)
+			(at 97.79 54.61 0)
 			(effects
 				(font
@@
 		)
 		(property "Footprint" ""
-			(at 94.742 50.8 90)
+			(at 94.742 53.34 90)
 			(effects
 				(font
@@
 		)
 		(property "Datasheet" "~"
-			(at 96.52 50.8 0)
+			(at 96.52 53.34 0)
 			(effects
 				(font
@@
 		)
 		(property "Description" "Resistor"
-			(at 96.52 50.8 0)
+			(at 96.52 53.34 0)
 			(effects
 				(font
@@
 		(on_board yes)
 		(dnp no)
-		(property "Reference" "Q304"
+		(property "Reference" "Q305"
 			(at 154.94 92.71 0)
+			(do_not_autoplace yes)
 			(effects
 				(font
@@
 			(project "y_board"
 				(path "/b3bc71fd-0ca0-4281-9bf5-aadd2561d695/e0518060-d474-471b-9624-7dbd2316e9c6"
-					(reference "Q304")
+					(reference "Q305")
 					(unit 1)
 				)
@@
 					(unit 1)
 				)
+			)
+		)
+	)
+	(symbol
+		(lib_id "Device:R")
+		(at 109.22 31.75 0)
+		(unit 1)
+		(exclude_from_sim no)
+		(in_bom yes)
+		(on_board yes)
+		(dnp no)
+		(property "Reference" "R333"
+			(at 101.6 30.48 0)
+			(effects
+				(font
+					(size 1.27 1.27)
+				)
+				(justify left)
+			)
+		)
+		(property "Value" "1k"
+			(at 102.87 33.02 0)
+			(effects
+				(font
+					(size 1.27 1.27)
+				)
+				(justify left)
+			)
+		)
+		(property "Footprint" ""
+			(at 107.442 31.75 90)
+			(effects
+				(font
+					(size 1.27 1.27)
+				)
+				(hide yes)
+			)
+		)
+		(property "Datasheet" "~"
+			(at 109.22 31.75 0)
+			(effects
+				(font
+					(size 1.27 1.27)
+				)
+				(hide yes)
+			)
+		)
+		(property "Description" "Resistor"
+			(at 109.22 31.75 0)
+			(effects
+				(font
+					(size 1.27 1.27)
+				)
+				(hide yes)
+			)
+		)
+		(pin "1"
+		)
+		(pin "2"
+		)
+		(instances
+			(project "y_board"
+				(path "/b3bc71fd-0ca0-4281-9bf5-aadd2561d695/e0518060-d474-471b-9624-7dbd2316e9c6"
+					(reference "R333")
+					(unit 1)
+				)

Commit message: Finishing implementing output control
Connections:
- net OE_IC102 renamed OE
Changed lines of the file:
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@@
 		)
 	)
-	(global_label "OE_IC102"
+	(global_label "OE"
 		(shape passive)
 		(at 62.23 38.1 180)
@@
 		)
 		(property "Intersheetrefs" "${INTERSHEET_REFS}"
-			(at 51.4057 38.1 0)
+			(at 57.8766 38.1 0)
 			(effects
 				(font

Commit message: Implement Output Control
Parts:
- renumbered D4 to D301, IC401 to IC302, R9 to R233, R8 to R325
Connections:
- net I_DET_LEVEL_SEL_A: no longer names the net of C304.2, IC302.2 (IN1-), R309.2, R311.1, R320.1, ZD302.1 (K)
Changed lines of the file:
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@@
 	(wire
 		(pts
-			(xy 100.33 151.13) (xy 158.75 151.13)
-		)
-		(stroke
-			(width 0)
-			(type default)
-		)
-	)
-	(wire
-		(pts
 			(xy 226.06 115.57) (xy 215.9 115.57)
 		)
@@
 	(wire
 		(pts
-			(xy 158.75 151.13) (xy 158.75 129.54)
-		)
-		(stroke
-			(width 0)
-			(type default)
-		)
-	)
-	(wire
-		(pts
 			(xy 120.65 111.76) (xy 120.65 115.57)
 		)
@@
 		)
 	)
-	(global_label "I_DET_LEVEL_SEL_A"
-		(shape passive)
-		(at 100.33 151.13 180)
-		(fields_autoplaced yes)
-		(effects
-			(font
-				(size 1.27 1.27)
-			)
-			(justify right)
-		)
-		(property "Intersheetrefs" "${INTERSHEET_REFS}"
-			(at 80.6763 151.13 0)
-			(effects
-				(font
-					(size 1.27 1.27)
-				)
-				(justify right)
-				(hide yes)
-			)
-		)
-	)
 	(global_label "OE"
 		(shape passive)
@@
 		(on_board yes)
 		(dnp no)
-		(property "Reference" "R9"
+		(property "Reference" "R233"
 			(at 228.6 100.33 0)
 			(effects
@@
 			(project "y_board"
 				(path "/b3bc71fd-0ca0-4281-9bf5-aadd2561d695/e0518060-d474-471b-9624-7dbd2316e9c6"
-					(reference "R9")
+					(reference "R233")
 					(unit 1)
 				)
@@
 		(on_board yes)
 		(dnp no)
-		(property "Reference" "R8"
+		(property "Reference" "R325"
 			(at 200.66 72.39 0)
 			(effects
@@
 			(project "y_board"
 				(path "/b3bc71fd-0ca0-4281-9bf5-aadd2561d695/e0518060-d474-471b-9624-7dbd2316e9c6"
-					(reference "R8")
+					(reference "R325")
 					(unit 1)
 				)
@@
 		(on_board yes)
 		(dnp no)
-		(property "Reference" "D4"
+		(property "Reference" "D301"
 			(at 195.58 82.55 90)
 			(effects
@@
 			(project "y_board"
 				(path "/b3bc71fd-0ca0-4281-9bf5-aadd2561d695/e0518060-d474-471b-9624-7dbd2316e9c6"
-					(reference "D4")
+					(reference "D301")
 					(unit 1)
 				)
@@
 		(on_board yes)
 		(dnp no)
-		(property "Reference" "IC401"
+		(property "Reference" "IC302"
 			(at 204.47 119.38 0)
 			(effects
@@
 			(project "y_board"
 				(path "/b3bc71fd-0ca0-4281-9bf5-aadd2561d695/e0518060-d474-471b-9624-7dbd2316e9c6"
-					(reference "IC401")
+					(reference "IC302")
 					(unit 1)
 				)

Commit message: Finishing Y BOARD reverse engineering. Todo: Add reverse conduction and resistence to all output/input pins and refactor Z BOARD DRC
Other:
- note added: "VSC and VY (Part 3 of 3)"
Changed lines of the file:
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@@
 		)
 	)
-	(label "VSC and VY (Part 3 of 3)"
-		(at 190.5 22.86 180)
+	(text "VSC and VY (Part 3 of 3)"
+		(exclude_from_sim no)
+		(at 147.32 19.05 0)
 		(effects
 			(font
-				(face "KiCad Font")
 				(size 5 5)
-				(thickness 0.254)
+				(thickness 0.6)
 				(bold yes)
 				(italic yes)
 			)
-			(justify right bottom)
 		)
 	)

Commit message: Finishing reverse engineering Y BOARD
Changed lines of the file:
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@@
 	)
 	(global_label "OE"
-		(shape passive)
+		(shape output)
 		(at 62.23 38.1 180)
 		(fields_autoplaced yes)
@@
 		)
 		(property "Intersheetrefs" "${INTERSHEET_REFS}"
-			(at 57.8766 38.1 0)
+			(at 56.7653 38.1 0)
 			(effects
 				(font

Commit message: Adding SMD capacitor values in SetUp circuit block
Parts:
- C306: value C_Small -> 100nF
Changed lines of the file:
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@@
 		(dnp no)
 		(property "Reference" "C306"
-			(at 199.39 149.86 0)
+			(at 200.66 149.86 0)
 			(effects
 				(font
@@
 			)
 		)
-		(property "Value" "C_Small"
-			(at 190.5 149.8538 0)
+		(property "Value" "100nF"
+			(at 201.93 152.4 0)
 			(effects
 				(font
@@
 				)
 				(justify left)
-				(hide yes)
 			)
 		)

Commit message: Add values to SMD capacitors C305 and C401
Parts:
- C305: value C_Small -> 100nF
Changed lines of the file:
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@@
 		(dnp no)
 		(property "Reference" "C305"
-			(at 223.52 149.86 0)
+			(at 224.79 149.86 0)
 			(effects
 				(font
@@
 			)
 		)
-		(property "Value" "C_Small"
-			(at 214.63 149.8538 0)
+		(property "Value" "100nF"
+			(at 226.06 152.4 0)
 			(effects
 				(font
@@
 				)
 				(justify left)
-				(hide yes)
 			)
 		)
