File: TV_PLASMA/42PQ30R/y_board/vsc_and_vy_part3_of_3.kicad_sch (KiCad schematic)
At the start: 32 parts, among them IC303 EL817, Q302 Q_NPN_BCE, Q304 Q_SCR_KGA, Q305 NMOS

Commit message: Finishing implement reverse engineering
Parts:
- C309: value C_Small -> 1uF
Changed lines of the file:
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@@
 			)
 		)
-		(property "Value" "C_Small"
-			(at 102.87 99.0538 0)
+		(property "Value" "1uF"
+			(at 111.76 101.6 0)
 			(effects
 				(font
@@
 				)
 				(justify left)
-				(hide yes)
 			)
 		)

Commit message: Add missing resistors
Parts:
- removed Q302: Q_NPN_BCE, symbol Device:Q_NPN_BCE
- added Q302: Q_PNP_BCE, symbol Device:Q_PNP_BCE
Connections:
- net at R327.2, R330.1: now also Q302.3 (E)
- net at IC303.3, R325.1, R326.1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: now also Q302.1 (B)
- net at R328.1: now also Q302.2 (C)
Other:
- moved on the sheet: C309, R326, R327, R330

Commit message: Add circuit protection information
Other:
- note added: "ZD302: Abnormal ER_CON_monitor voltages (Shutdown): ER_CON< 43.6 V @ ER_CON_monitor < 3.97 V ER_CON > 130 V @ ER_CON_monitor> 130 V"
Changed lines of the file:
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@@
+		)
+	)
+	(text "ZD302:\n\nAbnormal ER_CON_monitor voltages (Shutdown):\n\nER_CON< 43.6 V @ ER_CON_monitor < 3.97 V\nER_CON > 130 V @ ER_CON_monitor> 130 V"
+		(exclude_from_sim no)
+		(at 111.76 151.13 0)
+		(effects
+			(font
+				(size 1.27 1.27)
+				(thickness 0.254)
+				(bold yes)
+			)
+			(justify left)
+		)
+	)
+	(label "ER_CON_monitor"
+		(at 137.16 128.27 0)
+		(effects
+			(font
+				(size 1.27 1.27)
+			)
+			(justify left bottom)
 		)
 	)

Commit message: Update Y-Board schematics and add Y-Board top detailed information
Other:
- note added: "ZD302: Abnormal ER_CON_monitor voltages (Shutdown): ER_CON < 43.6 V @ ER_CON_monitor < 3.97 V ER_CON > 130 V @ ER_CON_monitor > 11.8 V"
- note removed: "ZD302: Abnormal ER_CON_monitor voltages (Shutdown): ER_CON< 43.6 V @ ER_CON_monitor < 3.97 V ER_CON > 130 V @ ER_CON_monitor> 130 V"
Changed lines of the file:
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@@
 		)
 	)
-	(text "ZD302:\n\nAbnormal ER_CON_monitor voltages (Shutdown):\n\nER_CON< 43.6 V @ ER_CON_monitor < 3.97 V\nER_CON > 130 V @ ER_CON_monitor> 130 V"
+	(text "ZD302:\n\nAbnormal ER_CON_monitor voltages (Shutdown):\n\nER_CON < 43.6 V @ ER_CON_monitor < 3.97 V\nER_CON > 130 V @ ER_CON_monitor > 11.8 V"
 		(exclude_from_sim no)
 		(at 111.76 151.13 0)

Commit message: Finishing document detailed images
Parts:
- IC302: value ~ -> AS393M
Changed lines of the file:
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@@
 			)
 		)
-		(property "Value" "~"
+		(property "Value" "AS393M"
 			(at 203.835 102.87 0)
 			(effects
