File: TV_PLASMA/42PQ30R/y_board/vsc_and_vy.kicad_sch (KiCad schematic)
At the start: 44 parts, among them IC501 EL817, IC501 NCP1200D60, Q502 Q_NPN_BCE, Q505 NMOS, Q506 Q_NPN_BCE, Q507 Q_NPN_BCE, T501 Transformer_1P_2S

Commit message: Finishing VSC and VY supply
Connections:
- net 15VFY renamed 15VYF
Changed lines of the file:
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@@
 	)
 	(global_label "OE_IC102"
-		(shape input)
+		(shape passive)
 		(at 41.91 167.64 180)
 		(fields_autoplaced yes)
@@
 		)
 		(property "Intersheetrefs" "${INTERSHEET_REFS}"
-			(at 29.9744 167.64 0)
+			(at 31.0857 167.64 0)
 			(effects
 				(font
@@
 		)
 	)
-	(global_label "15VFY"
+	(global_label "15VYF"
 		(shape input)
 		(at 36.83 99.06 180)

Commit message: Finishing 15VF, 5VF and 15V power supply
Changed lines of the file:
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@@
+	)
+	(symbol
+		(lib_name "Transformer_1P_2S_1")
+		(lib_id "transformer_1p_2s_edited:Transformer_1P_2S")
+		(at 147.32 57.15 0)
+		(mirror y)
+		(unit 1)
+		(exclude_from_sim no)
+		(in_bom yes)
+		(on_board yes)
+		(dnp no)
+		(property "Reference" "T501"
+			(at 147.955 41.91 0)
+			(effects
+				(font
+					(size 1.27 1.27)
+				)
+			)
+		)
+		(property "Value" "Transformer_1P_2S"
+			(at 147.955 44.45 0)
+			(effects
+				(font
+					(size 1.27 1.27)
+				)
+				(hide yes)
+			)
+		)
+		(property "Footprint" ""
+			(at 147.32 57.15 0)
+			(effects
+				(font
+					(size 1.27 1.27)
+				)
+				(hide yes)
+			)
+		)
+		(property "Datasheet" "~"
+			(at 147.32 57.15 0)
+			(effects
+				(font
+					(size 1.27 1.27)
+				)
+				(hide yes)
+			)
+		)
+		(property "Description" "Transformer, single primary, dual secondary"
+			(at 147.32 57.15 0)
+			(effects
+				(font
+					(size 1.27 1.27)
+				)
+				(hide yes)
+			)
+		)
+		(pin "5"
+		)
+		(pin "1"
+		)
+		(pin "2"
+		)
+		(pin "6"
+		)
+		(pin "4"
+		)
+		(pin "3"
+		)
+		(instances
+			(project ""
+				(path "/b3bc71fd-0ca0-4281-9bf5-aadd2561d695/24722eec-b18f-4f1f-afe2-83a605a5bded"
+					(reference "T501")
+					(unit 1)
+				)
+			)
+		)
 	)
 	(symbol
@@
 					(unit 1)
 				)
-			)
-		)
-	)
-	(symbol
-		(lib_id "transformer_1p_2s_edited:Transformer_1P_2S")
-		(at 147.32 57.15 0)
-		(mirror y)
-		(unit 1)
-		(exclude_from_sim no)
-		(in_bom yes)
-		(on_board yes)
-		(dnp no)
-		(property "Reference" "T501"
-			(at 147.32 44.45 0)
-			(effects
-				(font
-					(size 1.27 1.27)
-				)
-			)
-		)
-		(property "Value" "Transformer_1P_2S"
-			(at 147.955 44.45 0)
-			(effects
-				(font
-					(size 1.27 1.27)
-				)
-				(hide yes)
-			)
-		)
-		(property "Footprint" ""
-			(at 147.32 57.15 0)
-			(effects
-				(font
-					(size 1.27 1.27)
-				)
-				(hide yes)
-			)
-		)
-		(property "Datasheet" "~"
-			(at 147.32 57.15 0)
-			(effects
-				(font
-					(size 1.27 1.27)
-				)
-				(hide yes)
-			)
-		)
-		(property "Description" "Transformer, single primary, dual secondary"
-			(at 147.32 57.15 0)
-			(effects
-				(font
-					(size 1.27 1.27)
-				)
-				(hide yes)
-			)
-		)
-		(pin "4"
-		)
-		(pin "6"
-		)
-		(pin "5"
-		)
-		(pin "1"
-		)
-		(pin "2"
-		)
-		(pin "3"
-		)
-		(instances
-			(project ""
-				(path "/b3bc71fd-0ca0-4281-9bf5-aadd2561d695/24722eec-b18f-4f1f-afe2-83a605a5bded"
-					(reference "T501")
-					(unit 1)
-				)

Commit message: Finishing implementing output control
Connections:
- net OE_IC102 renamed OE
Changed lines of the file:
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@@
 		)
 	)
-	(global_label "OE_IC102"
+	(global_label "OE"
 		(shape passive)
 		(at 41.91 167.64 180)
@@
 		)
 		(property "Intersheetrefs" "${INTERSHEET_REFS}"
-			(at 31.0857 167.64 0)
+			(at 37.5566 167.64 0)
 			(effects
 				(font

Commit message: Finishing Y BOARD reverse engineering. Todo: Add reverse conduction and resistence to all output/input pins and refactor Z BOARD DRC
Parts:
- added R526: 680, symbol Device:R
- R512: renamed from R524; value 22k -> 220k
- R524: value 22k -> 220k
- renumbered IC501 to IC502, R718 to R503
Connections:
- net at R525.2, R527.2, VR502.3: now also R526.2
- net at R524.2, VR502.1: now also R526.1
Other:
- note added: "VSC and VY (Part 1 of 3)"
- note added: "VY_ADJUST"
- moved on the sheet: R524
Changed lines of the file:
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@@
 		(color 0 0 0 0)
 	)
+	(junction
+		(at 45.72 123.19)
+		(diameter 0)
+		(color 0 0 0 0)
+	)
 	(wire
 		(pts
@@
 	(wire
 		(pts
+			(xy 29.21 127) (xy 29.21 123.19)
+		)
+		(stroke
+			(width 0)
+			(type default)
+		)
+	)
+	(wire
+		(pts
 			(xy 87.63 83.82) (xy 87.63 85.09)
 		)
@@
 	(wire
 		(pts
+			(xy 29.21 134.62) (xy 29.21 146.05)
+		)
+		(stroke
+			(width 0)
+			(type default)
+		)
+	)
+	(wire
+		(pts
 			(xy 247.65 121.92) (xy 237.49 121.92)
 		)
@@
 	(wire
 		(pts
-			(xy 45.72 123.19) (xy 45.72 128.27)
+			(xy 45.72 118.11) (xy 45.72 123.19)
 		)
 		(stroke
@@
 	(wire
 		(pts
+			(xy 45.72 123.19) (xy 45.72 128.27)
+		)
+		(stroke
+			(width 0)
+			(type default)
+		)
+	)
+	(wire
+		(pts
 			(xy 215.9 91.44) (xy 208.28 91.44)
 		)
@@
 	(wire
 		(pts
+			(xy 29.21 146.05) (xy 45.72 146.05)
+		)
+		(stroke
+			(width 0)
+			(type default)
+		)
+	)
+	(wire
+		(pts
 			(xy 208.28 86.36) (xy 228.6 86.36)
 		)
@@
 	(wire
 		(pts
-			(xy 45.72 60.96) (xy 45.72 115.57)
+			(xy 29.21 123.19) (xy 45.72 123.19)
+		)
+		(stroke
+			(width 0)
+			(type default)
+		)
+	)
+	(wire
+		(pts
+			(xy 45.72 60.96) (xy 45.72 110.49)
 		)
 		(stroke
@@
 		)
 	)
-	(label "VSC and VY (Part 1 of 3)"
-		(at 200.66 25.4 180)
+	(text "VY_ADJUST"
+		(exclude_from_sim no)
+		(at 54.61 129.54 0)
 		(effects
 			(font
-				(face "KiCad Font")
-				(size 5 5)
+				(size 1.27 1.27)
 				(thickness 0.254)
 				(bold yes)
 				(italic yes)
 			)
-			(justify right bottom)
 		)
 	)
-	(label "VY_ADJUST"
-		(at 33.02 137.16 0)
+	(text "VSC and VY (Part 1 of 3)"
+		(exclude_from_sim no)
+		(at 154.94 21.59 0)
 		(effects
 			(font
-				(size 1.27 1.27)
-				(thickness 0.254)
+				(size 5 5)
+				(thickness 0.6)
 				(bold yes)
 				(italic yes)
-				(color 9 1 255 1)
 			)
-			(justify left bottom)
 		)
 	)
@@
 	(symbol
 		(lib_id "Device:R")
+		(at 29.21 130.81 0)
+		(unit 1)
+		(exclude_from_sim no)
+		(in_bom yes)
+		(on_board yes)
+		(dnp no)
+		(property "Reference" "R526"
+			(at 30.48 129.54 0)
+			(effects
+				(font
+					(size 1.27 1.27)
+				)
+				(justify left)
+			)
+		)
+		(property "Value" "680"
+			(at 30.48 132.08 0)
+			(effects
+				(font
+					(size 1.27 1.27)
+				)
+				(justify left)
+			)
+		)
+		(property "Footprint" ""
+			(at 27.432 130.81 90)
+			(effects
+				(font
+					(size 1.27 1.27)
+				)
+				(hide yes)
+			)
+		)
+		(property "Datasheet" "~"
+			(at 29.21 130.81 0)
+			(effects
+				(font
+					(size 1.27 1.27)
+				)
+				(hide yes)
+			)
+		)
+		(property "Description" "Resistor"
+			(at 29.21 130.81 0)
+			(effects
+				(font
+					(size 1.27 1.27)
+				)
+				(hide yes)
+			)
+		)
+		(pin "1"
+		)
+		(pin "2"
+		)
+		(instances
+			(project "y_board"
+				(path "/b3bc71fd-0ca0-4281-9bf5-aadd2561d695/24722eec-b18f-4f1f-afe2-83a605a5bded"
+					(reference "R526")
+					(unit 1)
+				)
+			)
+		)
+	)
+	(symbol
+		(lib_id "Device:R")
 		(at 180.34 97.79 0)
 		(unit 1)
@@
 	(symbol
 		(lib_id "Device:R")
-		(at 45.72 119.38 0)
+		(at 45.72 114.3 0)
 		(unit 1)
 		(exclude_from_sim no)
@@
 		(dnp no)
 		(property "Reference" "R524"
-			(at 46.99 118.11 0)
+			(at 46.99 113.03 0)
 			(effects
 				(font
@@
 			)
 		)
-		(property "Value" "22k"
-			(at 46.99 120.65 0)
+		(property "Value" "220k"
+			(at 46.99 115.57 0)
 			(effects
 				(font
@@
 		)
 		(property "Footprint" ""
-			(at 43.942 119.38 90)
+			(at 43.942 114.3 90)
 			(effects
 				(font
@@
 		)
 		(property "Datasheet" "~"
-			(at 45.72 119.38 0)
+			(at 45.72 114.3 0)
 			(effects
 				(font
@@
 		)
 		(property "Description" "Resistor"
-			(at 45.72 119.38 0)
+			(at 45.72 114.3 0)
 			(effects
 				(font
@@
 		(on_board yes)
 		(dnp no)
-		(property "Reference" "R524"
+		(property "Reference" "R512"
 			(at 185.42 59.69 0)
 			(effects
@@
 			)
 		)
-		(property "Value" "22k"
+		(property "Value" "220k"
 			(at 185.42 62.23 0)
 			(effects
@@
 			(project "y_board"
 				(path "/b3bc71fd-0ca0-4281-9bf5-aadd2561d695/24722eec-b18f-4f1f-afe2-83a605a5bded"
-					(reference "R524")
+					(reference "R512")
 					(unit 1)
 				)
@@
 		(dnp no)
 		(fields_autoplaced yes)
-		(property "Reference" "IC501"
+		(property "Reference" "IC502"
 			(at 90.17 104.14 0)
 			(effects
@@
 			(project ""
 				(path "/b3bc71fd-0ca0-4281-9bf5-aadd2561d695/24722eec-b18f-4f1f-afe2-83a605a5bded"
-					(reference "IC501")
+					(reference "IC502")
 					(unit 1)
 				)
@@
 		(on_board yes)
 		(dnp no)
-		(property "Reference" "R718"
+		(property "Reference" "R503"
 			(at 193.04 54.61 90)
 			(effects
@@
 			(project "y_board"
 				(path "/b3bc71fd-0ca0-4281-9bf5-aadd2561d695/24722eec-b18f-4f1f-afe2-83a605a5bded"
-					(reference "R718")
+					(reference "R503")
 					(unit 1)
 				)

Commit message: Finishing reverse engineering Y BOARD
Changed lines of the file:
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@@
 	)
 	(global_label "OE"
-		(shape passive)
+		(shape input)
 		(at 41.91 167.64 180)
 		(fields_autoplaced yes)
@@
 		)
 		(property "Intersheetrefs" "${INTERSHEET_REFS}"
-			(at 37.5566 167.64 0)
+			(at 36.4453 167.64 0)
 			(effects
 				(font

Commit message: Add missing capacitor. Add measured SMD capacitor values
Parts:
- C501: value C_Small -> 1uF
- C518: value C_Small -> 10nF
Changed lines of the file:
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@@
 			)
 		)
-		(property "Value" "C_Small"
-			(at 106.68 104.1338 0)
-			(effects
-				(font
-					(size 1.27 1.27)
-				)
-				(justify left)
-				(hide yes)
+		(property "Value" "1uF"
+			(at 106.68 105.41 0)
+			(effects
+				(font
+					(size 1.27 1.27)
+				)
+				(justify left)
 			)
 		)
@@
 		(dnp no)
 		(property "Reference" "C518"
-			(at 44.45 171.45 0)
-			(effects
-				(font
-					(size 1.27 1.27)
-				)
-				(justify left)
-			)
-		)
-		(property "Value" "C_Small"
-			(at 43.18 172.7138 0)
-			(effects
-				(font
-					(size 1.27 1.27)
-				)
-				(justify left)
-				(hide yes)
-			)
-		)
+			(at 41.91 175.26 0)
+			(effects
+				(font
+					(size 1.27 1.27)
+				)
+				(justify left)
+			)
+		)
+		(property "Value" "10nF"
+			(at 41.91 177.8 0)
+			(effects
+				(font
+					(size 1.27 1.27)
+				)
+				(justify left)
+			)
+		)

Commit message: Adding missing components. Add missing SMD capacitor values
Parts:
- C506, C509, C510: value C_Small -> 1nF
- C552: value C_Small -> 1uF
Changed lines of the file:
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@@
 	)
 	(junction
-		(at 63.5 151.13)
-		(diameter 0)
-		(color 0 0 0 0)
-	)
-	(junction
-		(at 63.5 85.09)
-		(diameter 0)
-		(color 0 0 0 0)
-	)
-	(junction
 		(at 184.15 52.07)
 		(diameter 0)
@@
 	)
 	(junction
-		(at 63.5 146.05)
+		(at 45.72 60.96)
 		(diameter 0)
 		(color 0 0 0 0)
 	)
 	(junction
-		(at 45.72 60.96)
+		(at 162.56 68.58)
 		(diameter 0)
 		(color 0 0 0 0)
 	)
 	(junction
-		(at 162.56 68.58)
+		(at 62.23 85.09)
 		(diameter 0)
 		(color 0 0 0 0)
@@
 	)
 	(junction
+		(at 62.23 146.05)
+		(diameter 0)
+		(color 0 0 0 0)
+	)
+	(junction
 		(at 124.46 100.33)
 		(diameter 0)
@@
 		(color 0 0 0 0)
 	)
+	(junction
+		(at 62.23 151.13)
+		(diameter 0)
+		(color 0 0 0 0)
+	)
 	(wire
 		(pts
@@
 	(wire
 		(pts
-			(xy 58.42 146.05) (xy 63.5 146.05)
+			(xy 58.42 146.05) (xy 62.23 146.05)
 		)
 		(stroke
@@
 	(wire
 		(pts
+			(xy 62.23 151.13) (xy 73.66 151.13)
+		)
+		(stroke
+			(width 0)
+			(type default)
+		)
+	)
+	(wire
+		(pts
 			(xy 97.79 113.03) (xy 109.22 113.03)
 		)
@@
 	(wire
 		(pts
-			(xy 63.5 85.09) (xy 63.5 146.05)
+			(xy 62.23 85.09) (xy 62.23 146.05)
 		)
 		(stroke
@@
 	(wire
 		(pts
-			(xy 36.83 85.09) (xy 63.5 85.09)
+			(xy 36.83 85.09) (xy 62.23 85.09)
 		)
 		(stroke
@@
 	(wire
 		(pts
+			(xy 62.23 85.09) (xy 68.58 85.09)
+		)
+		(stroke
+			(width 0)
+			(type default)
+		)
+	)
+	(wire
+		(pts
 			(xy 124.46 167.64) (xy 124.46 100.33)
 		)
@@
 	(wire
 		(pts
-			(xy 58.42 151.13) (xy 63.5 151.13)
-		)
-		(stroke
-			(width 0)
-			(type default)
-		)
-	)
-	(wire
-		(pts
-			(xy 63.5 85.09) (xy 68.58 85.09)
+			(xy 58.42 151.13) (xy 62.23 151.13)
 		)
 		(stroke
@@
 	(wire
 		(pts
-			(xy 63.5 151.13) (xy 73.66 151.13)
-		)
-		(stroke
-			(width 0)
-			(type default)
-		)
-	)
-	(wire
-		(pts
 			(xy 101.6 99.06) (xy 109.22 99.06)
 		)
@@
 	(wire
 		(pts
-			(xy 63.5 146.05) (xy 63.5 151.13)
+			(xy 62.23 146.05) (xy 62.23 151.13)
 		)
 		(stroke
@@
 		(dnp no)
 		(property "Reference" "C510"
-			(at 90.17 124.46 0)
+			(at 92.71 119.38 0)
 			(effects
 				(font
@@
 			)
 		)
-		(property "Value" "C_Small"
-			(at 91.44 123.1962 0)
+		(property "Value" "1nF"
+			(at 92.71 121.92 0)
 			(effects
 				(font
@@
 				)
 				(justify left)
-				(hide yes)
 			)
 		)
@@
 		(dnp no)
 		(property "Reference" "C552"
-			(at 76.2 90.17 0)
+			(at 74.93 87.63 0)
 			(effects
 				(font
@@
 			)
 		)
-		(property "Value" "C_Small"
-			(at 66.04 90.1638 0)
+		(property "Value" "1uF"
+			(at 74.93 90.17 0)
 			(effects
 				(font
@@
 				)
 				(justify left)
-				(hide yes)
 			)
 		)
@@
 		(dnp no)
 		(property "Reference" "C509"
-			(at 69.85 110.49 0)
+			(at 69.85 111.76 0)
 			(effects
 				(font
@@
 			)
 		)
-		(property "Value" "C_Small"
-			(at 68.58 111.7538 0)
+		(property "Value" "1nF"
+			(at 68.58 114.3 0)
 			(effects
 				(font
@@
 				)
 				(justify left)
-				(hide yes)
 			)
 		)
@@
 		(dnp no)
 		(property "Reference" "C506"
-			(at 177.8 62.23 0)
+			(at 176.53 55.88 0)
 			(effects
 				(font
@@
 			)
 		)
-		(property "Value" "C_Small"
+		(property "Value" "1nF"
 			(at 176.53 58.4138 0)
 			(effects
@@
 				)
 				(justify left)
-				(hide yes)
 			)
 		)

Commit message: Add circuit protection information
Other:
- note added: "VY_A Range: 147.7 V ~ 180.7 V"
Changed lines of the file:
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@@
+		)
+	)
+	(text "VY_A\n\nRange: 147.7 V ~ 180.7 V"
+		(exclude_from_sim no)
+		(at 30.48 118.11 0)
+		(effects
+			(font
+				(size 1.27 1.27)
+			)
 		)
 	)
