File: TV_PLASMA/42PQ30R/y_board/vsc_and_vy.kicad_sch (KiCad schematic)
At the start: 45 parts, among them IC501 NCP1200D60, IC502 EL817, Q502 Q_NPN_BCE, Q505 NMOS, Q506 Q_NPN_BCE, Q507 Q_NPN_BCE, T501 Transformer_1P_2S

Commit message: Finishing document detailed images
Parts:
- IC504: value ~ -> E43A 813J30
Changed lines of the file:
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@@
 		(dnp no)
 		(property "Reference" "IC504"
-			(at 71.12 138.43 90)
+			(at 72.39 133.35 90)
 			(effects
 				(font
@@
 			)
 		)
-		(property "Value" "~"
-			(at 71.12 137.1599 90)
+		(property "Value" "E43A 813J30"
+			(at 87.63 138.43 90)
 			(effects
 				(font
@@
 				)
 				(justify right)
-				(hide yes)
 			)
 		)

Commit message: Fix components values
Parts:
- R525: value 6.2k -> 5.6k
Changed lines of the file:
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@@
 			)
 		)
-		(property "Value" "6.2k"
+		(property "Value" "5.6k"
 			(at 54.61 143.51 90)
 			(effects

Commit message: Update Power transistor names
Parts:
- IC501: value NCP1200D60 -> 200D PL00
- Q503: renamed from Q505; value NMOS -> 5N50C
Changed lines of the file:
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@@
 		(on_board yes)
 		(dnp no)
-		(property "Reference" "Q505"
+		(property "Reference" "Q503"
 			(at 160.02 81.28 0)
 			(effects
@@
 			)
 		)
-		(property "Value" "NMOS"
-			(at 158.75 80.0099 0)
-			(effects
-				(font
-					(size 1.27 1.27)
-				)
-				(justify left)
-				(hide yes)
+		(property "Value" "5N50C"
+			(at 160.02 83.82 0)
+			(effects
+				(font
+					(size 1.27 1.27)
+				)
+				(justify left)
 			)
 		)
@@
 			(project "y_board"
 				(path "/b3bc71fd-0ca0-4281-9bf5-aadd2561d695/24722eec-b18f-4f1f-afe2-83a605a5bded"
-					(reference "Q505")
+					(reference "Q503")
 					(unit 1)
 				)
@@
 		(dnp no)
 		(property "Reference" "IC501"
-			(at 201.93 101.6 0)
-			(effects
-				(font
-					(size 1.27 1.27)
-				)
-				(justify left)
-			)
-		)
-		(property "Value" "NCP1200D60"
-			(at 202.8541 81.28 0)
-			(effects
-				(font
-					(size 1.27 1.27)
-				)
-				(justify left)
-				(hide yes)
-			)
-		)
+			(at 204.47 81.28 0)
+			(effects
+				(font
+					(size 1.27 1.27)
+				)
+				(justify left)
+			)
+		)
+		(property "Value" "200D PL00"
+			(at 187.96 81.28 0)
+			(effects
+				(font
+					(size 1.27 1.27)
+				)
+				(justify left)
+			)
+		)
