File: TV_PLASMA/42PQ30R/y_board/input_control2.kicad_sch (KiCad schematic)
At the start: 12 parts, among them IC102 74AHC541

Commit message: Finishing implementing output control
Connections:
- net OE_IC102 renamed OE
Changed lines of the file:
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@@
 		)
 	)
-	(global_label "OE_IC102"
+	(global_label "OE"
 		(shape passive)
 		(at 59.69 121.92 180)
@@
 		)
 		(property "Intersheetrefs" "${INTERSHEET_REFS}"
-			(at 48.8657 121.92 0)
+			(at 55.3366 121.92 0)
 			(effects
 				(font

Commit message: Implement Output Control
Parts:
- renumbered R127 to R124
Changed lines of the file:
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@@
 		(on_board yes)
 		(dnp no)
-		(property "Reference" "R127"
+		(property "Reference" "R124"
 			(at 218.44 91.44 0)
 			(effects
@@
 			(project "y_board"
 				(path "/b3bc71fd-0ca0-4281-9bf5-aadd2561d695/2e163e02-5861-47f2-ba93-a2117974138d"
-					(reference "R127")
+					(reference "R124")
 					(unit 1)
 				)

Commit message: Finishing Y BOARD reverse engineering. Todo: Add reverse conduction and resistence to all output/input pins and refactor Z BOARD DRC
Other:
- note added: "Input Control (Part 2 of 3)"
Changed lines of the file:
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@@
 		)
 	)
-	(label "Input Control (Part 2 of 3)"
-		(at 196.85 25.4 180)
+	(text "Input Control (Part 2 of 3)"
+		(exclude_from_sim no)
+		(at 146.05 22.86 0)
 		(effects
 			(font
-				(face "KiCad Font")
 				(size 5 5)
-				(thickness 0.254)
+				(thickness 0.6)
 				(bold yes)
 				(italic yes)
 			)
-			(justify right bottom)
 		)
 	)

Commit message: Finishing reverse engineering Y BOARD
Changed lines of the file:
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@@
 	)
 	(global_label "OE"
-		(shape passive)
+		(shape input)
 		(at 59.69 121.92 180)
 		(fields_autoplaced yes)
@@
 		)
 		(property "Intersheetrefs" "${INTERSHEET_REFS}"
-			(at 55.3366 121.92 0)
+			(at 54.2253 121.92 0)
 			(effects
 				(font

Commit message: Add missing capacitor. Add measured SMD capacitor values
Parts:
- C102: value C_Small -> 1uF
- C104: value C_Small -> 1nF
- R111, R117, R123, R124, R125, R129, R143: value 4.2k -> 4.7k
Changed lines of the file:
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@@
 			)
 		)
-		(property "Value" "C_Small"
-			(at 87.63 58.4138 0)
-			(effects
-				(font
-					(size 1.27 1.27)
-				)
-				(justify left)
-				(hide yes)
+		(property "Value" "1uF"
+			(at 87.63 64.77 0)
+			(effects
+				(font
+					(size 1.27 1.27)
+				)
+				(justify left)
 			)
 		)
@@
 			)
 		)
-		(property "Value" "4.2k"
+		(property "Value" "4.7k"
 			(at 162.56 111.76 0)
 			(effects
@@
 			)
 		)
-		(property "Value" "C_Small"
-			(at 104.14 59.6838 0)
-			(effects
-				(font
-					(size 1.27 1.27)
-				)
-				(justify left)
-				(hide yes)
+		(property "Value" "1nF"
+			(at 113.03 64.77 0)
+			(effects
+				(font
+					(size 1.27 1.27)
+				)
+				(justify left)
 			)
 		)
@@
 			)
 		)
-		(property "Value" "4.2k"
+		(property "Value" "4.7k"
 			(at 189.23 127 0)
 			(effects
@@
 			)
 		)
-		(property "Value" "4.2k"
+		(property "Value" "4.7k"
 			(at 218.44 93.98 0)
 			(effects
@@
 			)
 		)
-		(property "Value" "4.2k"
+		(property "Value" "4.7k"
 			(at 224.79 107.95 0)
 			(effects
@@
 			)
 		)
-		(property "Value" "4.2k"
+		(property "Value" "4.7k"
 			(at 99.06 60.96 0)
 			(effects
@@
 		(dnp no)
 		(property "Reference" "R123"
-			(at 210.82 76.2 0)
-			(effects
-				(font
-					(size 1.27 1.27)
-				)
-				(justify left)
-			)
-		)
-		(property "Value" "4.2k"
-			(at 210.82 78.74 0)
+			(at 201.93 76.2 0)
+			(effects
+				(font
+					(size 1.27 1.27)
+				)
+				(justify left)
+			)
+		)
+		(property "Value" "4.7k"
+			(at 203.2 78.74 0)
 			(effects
 				(font
@@
 			)
 		)
-		(property "Value" "4.2k"
+		(property "Value" "4.7k"
 			(at 162.56 128.27 0)
 			(effects

Commit message: Finishing document detailed images
Parts:
- IC102: value 74AHC541 -> VHC T541A
Changed lines of the file:
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@@
 		(on_board yes)
 		(dnp no)
-		(fields_autoplaced yes)
 		(property "Reference" "IC102"
 			(at 138.0841 77.47 0)
@@
 			)
 		)
-		(property "Value" "74AHC541"
-			(at 138.0841 77.47 0)
+		(property "Value" "VHC T541A"
+			(at 137.16 113.03 0)
 			(effects
 				(font
@@
 				)
 				(justify left)
-				(hide yes)
 			)
 		)
