File: TV_PLASMA/42PQ30R/y_board/output_control.kicad_sch (KiCad schematic)
At the start: 11 parts

Commit message: Finishing Y BOARD reverse engineering. Todo: Add reverse conduction and resistence to all output/input pins and refactor Z BOARD DRC
Other:
- note added: "OUPUT CONTROL (Part 1 of 4)"
Changed lines of the file:
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@@
 		(rev "1.0")
 		(comment 1 "Author: Fábio Pereira da Silva")
-		(comment 2 "Output Control (Part 1 of 3)")
+		(comment 2 "Output Control (Part 1 of 4)")
 	)
 	(junction
@@
 		)
 	)
-	(label "OUPUT CONTROL (Part 1 of 3)"
-		(at 194.31 26.67 180)
+	(text "OUPUT CONTROL (Part 1 of 4)"
+		(exclude_from_sim no)
+		(at 147.32 22.86 0)
 		(effects
 			(font
-				(face "KiCad Font")
 				(size 5 5)
-				(thickness 0.254)
+				(thickness 0.6)
 				(bold yes)
 				(italic yes)
 			)
-			(justify right bottom)
-		)
-	)
+		)
+	)

Commit message: Add values to SMD capacitors C305 and C401
Parts:
- C401: value C_Small -> 1uF
Changed lines of the file:
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@@
 		(dnp no)
 		(property "Reference" "C401"
-			(at 176.53 107.95 0)
+			(at 186.69 106.68 0)
 			(effects
 				(font
@@
 			)
 		)
-		(property "Value" "C_Small"
+		(property "Value" "1uF"
 			(at 186.69 110.4962 0)
 			(effects
@@
 				)
 				(justify left)
-				(hide yes)
 			)
 		)

Commit message: Finishing document detailed images
Parts:
- IC401: value ~ -> AS393M
Changed lines of the file:
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@@
 			)
 		)
-		(property "Value" "~"
+		(property "Value" "AS393M"
 			(at 158.115 95.25 0)
 			(effects
