File: TV_PLASMA/42PQ30R/y_board/5VF_15VF_15V.kicad_sch (KiCad schematic)
At the start: 34 parts, among them IC503 NMOS, IC505 L7805, IC507 L7818, IC508 L7805, Q504 Q_NPN_BCE, T502 Transformer_1P_2S

Commit message: Finishing Y BOARD reverse engineering. Todo: Add reverse conduction and resistence to all output/input pins and refactor Z BOARD DRC
Parts:
- added C719, C722: 1nF/1kV, symbol Device:C_Small
- renumbered R533 to R532, R536 to R535
Connections:
- net 15VF: now also IC507.3 (OUT); no longer IC507.1 (IN)
- net 5VF: now also IC508.3 (OUT); no longer IC508.1 (IN)
- net Earth: now also C719.2, C722.2
- net Y_OUT: now also C719.1, C722.1
- net at C519.1, D508.1 (K), D510.1 (K): now also IC507.1 (IN); no longer IC507.3 (OUT)
- net at C520.1, D509.1 (K), D511.1 (K): now also IC508.1 (IN); no longer IC508.3 (OUT)
- net OE_IC103 renamed OE
Other:
- note added: "5VF, 15VF and 15V Supply"

Commit message: Finishing reverse engineering Y BOARD
Changed lines of the file:
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@@
 	)
 	(global_label "OE"
-		(shape passive)
+		(shape input)
 		(at 36.83 134.62 180)
 		(fields_autoplaced yes)
@@
 		)
 		(property "Intersheetrefs" "${INTERSHEET_REFS}"
-			(at 32.4766 134.62 0)
+			(at 31.3653 134.62 0)
 			(effects
 				(font

Commit message: Insert SMD capacitors measured values
Parts:
- C219: value C_Small -> 1uF
Changed lines of the file:
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@@
 		(dnp no)
 		(property "Reference" "C219"
-			(at 54.61 74.93 0)
+			(at 53.34 69.85 0)
 			(effects
 				(font
@@
 			)
 		)
-		(property "Value" "C_Small"
-			(at 63.5 73.6662 0)
+		(property "Value" "1uF"
+			(at 54.61 72.39 0)
 			(effects
 				(font
@@
 				)
 				(justify left)
-				(hide yes)
 			)
 		)

Commit message: Add values to SMD capacitors in Set Down circuit. Add missing capacitors
Parts:
- added C308: 1uF, symbol Device:C_Small
Connections:
- net 15V: now also C308.1
- net Earth: now also C308.2
Changed lines of the file:
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@@
+	)
+	(junction
+		(at 204.47 50.8)
+		(diameter 0)
+		(color 0 0 0 0)
 	)
 	(junction
@@
 	(wire
 		(pts
+			(xy 204.47 50.8) (xy 219.71 50.8)
+		)
+		(stroke
+			(width 0)
+			(type default)
+		)
+	)
+	(wire
+		(pts
 			(xy 191.77 76.2) (xy 204.47 76.2)
 		)
@@
 	(wire
 		(pts
-			(xy 34.29 50.8) (xy 219.71 50.8)
+			(xy 34.29 50.8) (xy 204.47 50.8)
 		)
 		(stroke
@@
 	(wire
 		(pts
+			(xy 204.47 55.88) (xy 204.47 50.8)
+		)
+		(stroke
+			(width 0)
+			(type default)
+		)
+	)
+	(wire
+		(pts
 			(xy 205.74 132.08) (xy 208.28 132.08)
 		)
@@
 		(pts
 			(xy 118.11 81.28) (xy 110.49 81.28)
+		)
+		(stroke
+			(width 0)
+			(type default)
+		)
+	)
+	(wire
+		(pts
+			(xy 204.47 60.96) (xy 204.47 66.04)
 		)
 		(stroke
@@
 	(symbol
 		(lib_id "Device:C_Small")
+		(at 204.47 58.42 0)
+		(unit 1)
+		(exclude_from_sim no)
+		(in_bom yes)
+		(on_board yes)
+		(dnp no)
+		(property "Reference" "C308"
+			(at 207.01 57.15 0)
+			(effects
+				(font
+					(size 1.27 1.27)
+				)
+				(justify left)
+			)
+		)
+		(property "Value" "1uF"
+			(at 207.01 59.6962 0)
+			(effects
+				(font
+					(size 1.27 1.27)
+				)
+				(justify left)
+			)
+		)
+		(property "Footprint" ""
+			(at 204.47 58.42 0)
+			(effects
+				(font
+					(size 1.27 1.27)
+				)
+				(hide yes)
+			)
+		)
+		(property "Datasheet" "~"
+			(at 204.47 58.42 0)
+			(effects
+				(font
+					(size 1.27 1.27)
+				)
+				(hide yes)
+			)
+		)
+		(property "Description" "Unpolarized capacitor, small symbol"
+			(at 204.47 58.42 0)
+			(effects
+				(font
+					(size 1.27 1.27)
+				)
+				(hide yes)
+			)
+		)
+		(pin "2"
+		)
+		(pin "1"
+		)
+		(instances
+			(project "y_board"
+				(path "/b3bc71fd-0ca0-4281-9bf5-aadd2561d695/76b17981-32d8-4a0e-82cc-bb657e39681a"
+					(reference "C308")
+					(unit 1)
+				)
+			)
+		)
+	)
+	(symbol
+		(lib_id "Device:C_Small")
 		(at 68.58 113.03 0)
 		(unit 1)
@@
 					(unit 1)
 				)
+			)
+		)
+	)
+	(symbol
+		(lib_id "power:Earth")
+		(at 204.47 66.04 0)
+		(unit 1)
+		(exclude_from_sim no)
+		(in_bom yes)
+		(on_board yes)
+		(dnp no)
+		(fields_autoplaced yes)
+		(property "Reference" "#PWR41"
+			(at 204.47 72.39 0)
+			(effects
+				(font
+					(size 1.27 1.27)
+				)
+				(hide yes)
+			)
+		)
+		(property "Value" "Earth"
+			(at 204.47 71.12 0)
+			(effects
+				(font
+					(size 1.27 1.27)
+				)
+				(hide yes)
+			)
+		)
+		(property "Footprint" ""
+			(at 204.47 66.04 0)
+			(effects
+				(font
+					(size 1.27 1.27)
+				)
+				(hide yes)
+			)
+		)
+		(property "Datasheet" "~"
+			(at 204.47 66.04 0)
+			(effects
+				(font
+					(size 1.27 1.27)
+				)
+				(hide yes)
+			)
+		)
+		(property "Description" "Power symbol creates a global label with name \"Earth\""
+			(at 204.47 66.04 0)
+			(effects
+				(font
+					(size 1.27 1.27)
+				)
+				(hide yes)
+			)
+		)
+		(pin "1"
+		)
+		(instances
+			(project "y_board"
+				(path "/b3bc71fd-0ca0-4281-9bf5-aadd2561d695/76b17981-32d8-4a0e-82cc-bb657e39681a"
+					(reference "#PWR41")
+					(unit 1)
+				)

Commit message: Add missing capacitor. Add measured SMD capacitor values
Parts:
- added C515: 220nF, symbol Device:C_Small
- C513, C514: value C_Small -> 1uF
- C517: value C_Small -> 100nF
Connections:
- net Earth: now also C515.2
- net at IC506.7 (CTL/SS), Q504.2 (C), R530.1: now also C515.1
Other:
- moved on the sheet: Q504, R533, R534
Changed lines of the file:
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@@
 	)
 	(junction
+		(at 171.45 149.86)
+		(diameter 0)
+		(color 0 0 0 0)
+	)
+	(junction
 		(at 135.89 81.28)
 		(diameter 0)
@@
 	)
 	(junction
-		(at 160.02 134.62)
+		(at 142.24 134.62)
 		(diameter 0)
 		(color 0 0 0 0)
@@
 	)
 	(junction
+		(at 171.45 115.57)
+		(diameter 0)
+		(color 0 0 0 0)
+	)
+	(junction
 		(at 118.11 81.28)
 		(diameter 0)
@@
 	)
 	(junction
-		(at 173.99 149.86)
+		(at 156.21 149.86)
 		(diameter 0)
 		(color 0 0 0 0)
@@
 	(wire
 		(pts
-			(xy 232.41 115.57) (xy 173.99 115.57)
+			(xy 232.41 115.57) (xy 171.45 115.57)
 		)
 		(stroke
@@
 	(wire
 		(pts
-			(xy 160.02 149.86) (xy 173.99 149.86)
+			(xy 142.24 149.86) (xy 156.21 149.86)
 		)
 		(stroke
@@
 	(wire
 		(pts
-			(xy 160.02 146.05) (xy 160.02 149.86)
+			(xy 142.24 146.05) (xy 142.24 149.86)
 		)
 		(stroke
@@
 	(wire
 		(pts
+			(xy 156.21 115.57) (xy 171.45 115.57)
+		)
+		(stroke
+			(width 0)
+			(type default)
+		)
+	)
+	(wire
+		(pts
 			(xy 128.27 104.14) (xy 128.27 91.44)
 		)
@@
 	(wire
 		(pts
-			(xy 173.99 149.86) (xy 190.5 149.86)
+			(xy 156.21 149.86) (xy 171.45 149.86)
 		)
 		(stroke
@@
 	(wire
 		(pts
-			(xy 149.86 134.62) (xy 160.02 134.62)
+			(xy 132.08 134.62) (xy 142.24 134.62)
 		)
 		(stroke
@@
 	(wire
 		(pts
-			(xy 36.83 134.62) (xy 142.24 134.62)
+			(xy 36.83 134.62) (xy 124.46 134.62)
 		)
 		(stroke
@@
 	(wire
 		(pts
-			(xy 160.02 134.62) (xy 160.02 138.43)
+			(xy 142.24 134.62) (xy 142.24 138.43)
 		)
 		(stroke
@@
 	(wire
 		(pts
-			(xy 160.02 134.62) (xy 166.37 134.62)
+			(xy 142.24 134.62) (xy 148.59 134.62)
 		)
 		(stroke
@@
 	(wire
 		(pts
+			(xy 171.45 149.86) (xy 190.5 149.86)
+		)
+		(stroke
+			(width 0)
+			(type default)
+		)
+	)
+	(wire
+		(pts
 			(xy 229.87 86.36) (xy 234.95 86.36)
 		)
@@
 	(wire
 		(pts
+			(xy 171.45 134.62) (xy 171.45 149.86)
+		)
+		(stroke
+			(width 0)
+			(type default)
+		)
+	)
+	(wire
+		(pts
 			(xy 247.65 92.71) (xy 247.65 76.2)
 		)
@@
 	(wire
 		(pts
+			(xy 171.45 115.57) (xy 171.45 129.54)
+		)
+		(stroke
+			(width 0)
+			(type default)
+		)
+	)
+	(wire
+		(pts
 			(xy 114.3 91.44) (xy 118.11 91.44)
 		)
@@
 	(wire
 		(pts
-			(xy 173.99 139.7) (xy 173.99 149.86)
+			(xy 156.21 139.7) (xy 156.21 149.86)
 		)
 		(stroke
@@
 	(wire
 		(pts
-			(xy 173.99 115.57) (xy 173.99 129.54)
+			(xy 156.21 115.57) (xy 156.21 129.54)
 		)
 		(stroke
@@
 		(dnp no)
 		(property "Reference" "C513"
-			(at 184.15 143.51 0)
+			(at 184.15 138.43 0)
 			(effects
 				(font
@@
 			)
 		)
-		(property "Value" "C_Small"
-			(at 193.04 142.2462 0)
+		(property "Value" "1uF"
+			(at 184.15 140.97 0)
 			(effects
 				(font
@@
 				)
 				(justify left)
-				(hide yes)
 			)
 		)
@@
 	(symbol
 		(lib_id "Device:Q_NPN_BCE")
-		(at 171.45 134.62 0)
+		(at 153.67 134.62 0)
 		(unit 1)
 		(exclude_from_sim no)
@@
 		(dnp no)
 		(property "Reference" "Q504"
-			(at 176.53 134.62 0)
+			(at 158.75 134.62 0)
 			(effects
 				(font
@@
 		)
 		(property "Value" "Q_NPN_BCE"
-			(at 176.53 135.8899 0)
+			(at 158.75 135.8899 0)
 			(effects
 				(font
@@
 		)
 		(property "Footprint" ""
-			(at 176.53 132.08 0)
+			(at 158.75 132.08 0)
 			(effects
 				(font
@@
 		)
 		(property "Datasheet" "~"
-			(at 171.45 134.62 0)
+			(at 153.67 134.62 0)
 			(effects
 				(font
@@
 		)
 		(property "Description" "NPN transistor, base/collector/emitter"
-			(at 171.45 134.62 0)
+			(at 153.67 134.62 0)
 			(effects
 				(font
@@
 		(dnp no)
 		(property "Reference" "C517"
-			(at 256.54 125.73 90)
+			(at 256.54 123.19 90)
 			(effects
 				(font
@@
 			)
 		)
-		(property "Value" "C_Small"
-			(at 255.2762 127 0)
+		(property "Value" "100nF"
+			(at 257.81 125.73 90)
 			(effects
 				(font
@@
 				)
 				(justify left)
-				(hide yes)
 			)
 		)
@@
 			)
 		)
-		(property "Value" "C_Small"
-			(at 208.28 144.7862 0)
+		(property "Value" "1uF"
+			(at 208.28 147.32 0)
 			(effects
 				(font
@@
 				)
 				(justify left)
-				(hide yes)
 			)
 		)
@@
 	(symbol
 		(lib_id "Device:R")
-		(at 160.02 142.24 180)
+		(at 142.24 142.24 180)
 		(unit 1)
 		(exclude_from_sim no)
@@
 		(dnp no)
 		(property "Reference" "R534"
-			(at 167.64 140.97 0)
+			(at 149.86 140.97 0)
 			(effects
 				(font
@@
 		)
 		(property "Value" "22k"
-			(at 166.37 143.51 0)
+			(at 148.59 143.51 0)
 			(effects
 				(font
@@
 		)
 		(property "Footprint" ""
-			(at 161.798 142.24 90)
+			(at 144.018 142.24 90)
 			(effects
 				(font
@@
 		)
 		(property "Datasheet" "~"
-			(at 160.02 142.24 0)
+			(at 142.24 142.24 0)
 			(effects
 				(font
@@
 		)
 		(property "Description" "Resistor"
-			(at 160.02 142.24 0)
+			(at 142.24 142.24 0)
 			(effects
 				(font
@@
 	)
 	(symbol
+		(lib_id "Device:C_Small")
+		(at 171.45 132.08 0)
+		(unit 1)
+		(exclude_from_sim no)
+		(in_bom yes)
+		(on_board yes)
+		(dnp no)
+		(property "Reference" "C515"
+			(at 175.26 130.81 0)
+			(effects
+				(font
+					(size 1.27 1.27)
+				)
+				(justify left)
+			)
+		)
+		(property "Value" "220nF"
+			(at 175.26 133.35 0)
+			(effects
+				(font
+					(size 1.27 1.27)
+				)
+				(justify left)
+			)
+		)
+		(property "Footprint" ""
+			(at 171.45 132.08 0)
+			(effects
+				(font
+					(size 1.27 1.27)
+				)
+				(hide yes)
+			)
+		)
+		(property "Datasheet" "~"
+			(at 171.45 132.08 0)
+			(effects
+				(font
+					(size 1.27 1.27)
+				)
+				(hide yes)
+			)
+		)
+		(property "Description" "Unpolarized capacitor, small symbol"
+			(at 171.45 132.08 0)
+			(effects
+				(font
+					(size 1.27 1.27)
+				)
+				(hide yes)
+			)
+		)
+		(pin "2"
+		)
+		(pin "1"
+		)
+		(instances
+			(project "y_board"
+				(path "/b3bc71fd-0ca0-4281-9bf5-aadd2561d695/76b17981-32d8-4a0e-82cc-bb657e39681a"
+					(reference "C515")
+					(unit 1)
+				)
+			)
+		)
+	)
+	(symbol
 		(lib_id "Device:R")
-		(at 146.05 134.62 270)
+		(at 128.27 134.62 270)
 		(unit 1)
 		(exclude_from_sim no)
@@
 		(dnp no)
 		(property "Reference" "R533"
-			(at 143.51 137.16 90)
+			(at 125.73 137.16 90)
 			(effects
 				(font
@@
 		)
 		(property "Value" "22k"
-			(at 143.51 139.7 90)
+			(at 125.73 139.7 90)
 			(effects
 				(font
@@
 		)
 		(property "Footprint" ""
-			(at 146.05 132.842 90)
+			(at 128.27 132.842 90)
 			(effects
 				(font
@@
 		)
 		(property "Datasheet" "~"
-			(at 146.05 134.62 0)
+			(at 128.27 134.62 0)
 			(effects
 				(font
@@
 		)
 		(property "Description" "Resistor"
-			(at 146.05 134.62 0)
+			(at 128.27 134.62 0)
 			(effects
 				(font

Commit message: Update capacitor values
Parts:
- C307: value C_Small -> 1uF
Changed lines of the file:
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@@
 		(dnp no)
 		(property "Reference" "C307"
-			(at 82.55 99.06 0)
+			(at 82.55 93.98 0)
 			(effects
 				(font
@@
 			)
 		)
-		(property "Value" "C_Small"
-			(at 91.44 97.7962 0)
+		(property "Value" "1uF"
+			(at 82.55 96.52 0)
 			(effects
 				(font
@@
 				)
 				(justify left)
-				(hide yes)
 			)
 		)

Commit message: Finishing document detailed images
Parts:
- IC506: value ~ -> D97 63 SJ
- IC508: value L7805 -> AS7805A
Changed lines of the file:
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@@
 		(dnp no)
 		(property "Reference" "IC506"
-			(at 218.44 119.38 0)
-			(effects
-				(font
-					(size 1.27 1.27)
-				)
-			)
-		)
-		(property "Value" "~"
+			(at 217.17 116.84 0)
+			(effects
+				(font
+					(size 1.27 1.27)
+				)
+			)
+		)
+		(property "Value" "D97 63 SJ"
 			(at 217.805 119.38 0)
 			(effects
@@
 			)
 		)
-		(property "Value" "L7805"
-			(at 77.47 63.5 0)
-			(effects
-				(font
-					(size 1.27 1.27)
-				)
-				(hide yes)
-			)
-		)
+		(property "Value" "AS7805A"
+			(at 82.55 74.93 0)
+			(effects
+				(font
+					(size 1.27 1.27)
+				)
+			)
+		)

Commit message: Update Power transistor names
Parts:
- IC503: value NMOS -> IR P919H
Changed lines of the file:
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@@
 			)
 		)
-		(property "Value" "NMOS"
-			(at 180.34 99.0599 0)
+		(property "Value" "IR P919H"
+			(at 180.34 100.33 0)
 			(effects
 				(font
@@
 				)
 				(justify left)
-				(hide yes)
 			)
 		)
