File: TV_PLASMA/42PQ30R/x_board/z_ctrl.kicad_sch (KiCad schematic)
At the start: 16 parts, among them IC1 VHCT541A

Commit message: Fix some Z-BOARD DRC
Parts:
- renumbered R38 to R28
Other:
- note added: "Z CONTROL"
Changed lines of the file:
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@@
 		)
 	)
-	(label "Z CONTROL"
-		(at 161.29 29.21 180)
+	(text "Z CONTROL"
+		(exclude_from_sim no)
+		(at 149.86 24.13 0)
 		(effects
 			(font
-				(face "KiCad Font")
 				(size 5 5)
 				(thickness 0.254)
@@
 				(italic yes)
 			)
-			(justify right bottom)
 		)
 	)
@@
 		(on_board yes)
 		(dnp no)
-		(property "Reference" "R38"
+		(property "Reference" "R28"
 			(at 118.11 133.35 90)
 			(effects
@@
 			(project "x_board"
 				(path "/5140f788-2f35-4c22-8e35-55ece5960fbd/df0afd2f-f090-478b-8167-213732ec1fbd"
-					(reference "R38")
-					(unit 1)
-				)
+					(reference "R28")
+					(unit 1)
+				)
