File: TV_PLASMA/42PQ30R/x_board/z_protection.kicad_sch (KiCad schematic)
At the start: 13 parts, among them IC31 VHC08

Commit message: Fix some Z-BOARD DRC
Parts:
- removed R312, R313: 100, symbol Device:R_Small
Connections:
- net Z_SUS_DOWN_5V: now also IC31.3 (Y1)
- net Z_SUS_UP_5V: now also IC31.6 (Y2)
Other:
- note added: "Z PROTECTION"
Changed lines of the file:
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@@
 	(wire
 		(pts
-			(xy 118.11 142.24) (xy 105.41 142.24)
+			(xy 105.41 142.24) (xy 208.28 142.24)
 		)
 		(stroke
@@
 	(wire
 		(pts
-			(xy 118.11 134.62) (xy 111.76 134.62)
+			(xy 111.76 134.62) (xy 208.28 134.62)
 		)
 		(stroke
@@
 	(wire
 		(pts
-			(xy 123.19 134.62) (xy 208.28 134.62)
-		)
-		(stroke
-			(width 0)
-			(type default)
-		)
-	)
-	(wire
-		(pts
 			(xy 190.5 95.25) (xy 190.5 97.79)
 		)
@@
 	(wire
 		(pts
-			(xy 123.19 142.24) (xy 208.28 142.24)
-		)
-		(stroke
-			(width 0)
-			(type default)
-		)
-	)
-	(wire
-		(pts
 			(xy 135.89 77.47) (xy 124.46 77.47)
 		)
@@
 		)
 	)
-	(label "Z PROTECTION"
-		(at 166.37 26.67 180)
+	(text "Z PROTECTION"
+		(exclude_from_sim no)
+		(at 139.7 22.86 0)
 		(effects
 			(font
-				(face "KiCad Font")
 				(size 5 5)
 				(thickness 0.254)
@@
 				(italic yes)
 			)
-			(justify right bottom)
 		)
 	)
@@
 				(justify left)
 				(hide yes)
-			)
-		)
-	)
-	(symbol
-		(lib_id "Device:R_Small")
-		(at 120.65 142.24 90)
-		(unit 1)
-		(exclude_from_sim no)
-		(in_bom yes)
-		(on_board yes)
-		(dnp no)
-		(property "Reference" "R313"
-			(at 120.65 144.78 90)
-			(effects
-				(font
-					(size 1.27 1.27)
-				)
-			)
-		)
-		(property "Value" "100"
-			(at 120.65 147.32 90)
-			(effects
-				(font
-					(size 1.27 1.27)
-				)
-			)
-		)
-		(property "Footprint" ""
-			(at 120.65 142.24 0)
-			(effects
-				(font
-					(size 1.27 1.27)
-				)
-				(hide yes)
-			)
-		)
-		(property "Datasheet" "~"
-			(at 120.65 142.24 0)
-			(effects
-				(font
-					(size 1.27 1.27)
-				)
-				(hide yes)
-			)
-		)
-		(property "Description" "Resistor, small symbol"
-			(at 120.65 142.24 0)
-			(effects
-				(font
-					(size 1.27 1.27)
-				)
-				(hide yes)
-			)
-		)
-		(pin "1"
-		)
-		(pin "2"
-		)
-		(instances
-			(project "x_board"
-				(path "/5140f788-2f35-4c22-8e35-55ece5960fbd/b3bb9483-a345-4909-963c-15baac620070"
-					(reference "R313")
-					(unit 1)
-				)
 			)
 		)
@@
 					(unit 1)
 				)
-			)
-		)
-	)
-	(symbol
-		(lib_id "Device:R_Small")
-		(at 120.65 134.62 90)
-		(unit 1)
-		(exclude_from_sim no)
-		(in_bom yes)
-		(on_board yes)
-		(dnp no)
-		(property "Reference" "R312"
-			(at 120.65 129.54 90)
-			(effects
-				(font
-					(size 1.27 1.27)
-				)
-			)
-		)
-		(property "Value" "100"
-			(at 120.65 132.08 90)
-			(effects
-				(font
-					(size 1.27 1.27)
-				)
-			)
-		)
-		(property "Footprint" ""
-			(at 120.65 134.62 0)
-			(effects
-				(font
-					(size 1.27 1.27)
-				)
-				(hide yes)
-			)
-		)
-		(property "Datasheet" "~"
-			(at 120.65 134.62 0)
-			(effects
-				(font
-					(size 1.27 1.27)
-				)
-				(hide yes)
-			)
-		)
-		(property "Description" "Resistor, small symbol"
-			(at 120.65 134.62 0)
-			(effects
-				(font
-					(size 1.27 1.27)
-				)
-				(hide yes)
-			)
-		)
-		(pin "1"
-		)
-		(pin "2"
-		)
-		(instances
-			(project "x_board"
-				(path "/5140f788-2f35-4c22-8e35-55ece5960fbd/b3bb9483-a345-4909-963c-15baac620070"
-					(reference "R312")
-					(unit 1)
-				)
