File: TV_PLASMA/42PQ30R/x_board/x_board.kicad_sch (KiCad schematic)
At the start: 9 parts

Commit message: Implemented Z ENERGY RECOVER UP/DOWN
Other:
- added sheet Z_ER_UP_AND_Z_ER_DOWN (z_er_up_and_z_er_dn.kicad_sch)
Changed lines of the file:
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@@
+		)
+	)
+	(sheet
+		(at -34.29 44.45)
+		(size 24.13 16.51)
+		(fields_autoplaced yes)
+		(stroke
+			(width 0.1524)
+			(type solid)
+		)
+		(fill
+			(color 0 0 0 0.0000)
+		)
+		(property "Sheetname" "Z_ER_UP_AND_Z_ER_DOWN"
+			(at -34.29 43.7384 0)
+			(effects
+				(font
+					(size 1.27 1.27)
+				)
+				(justify left bottom)
+			)
+		)
+		(property "Sheetfile" "z_er_up_and_z_er_dn.kicad_sch"
+			(at -34.29 61.5446 0)
+			(effects
+				(font
+					(size 1.27 1.27)
+				)
+				(justify left top)
+			)
+		)
+		(instances
+			(project "x_board"
+				(path "/5140f788-2f35-4c22-8e35-55ece5960fbd"
+					(page "3")
+				)
+			)
 		)
 	)

Commit message: Implement VZB and correct some Y BOARD
Other:
- added sheet VZB (vzb.kicad_sch)
Changed lines of the file:
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@@
 	)
 	(sheet
-		(at -34.29 44.45)
+		(at -36.83 31.75)
 		(size 24.13 16.51)
 		(fields_autoplaced yes)
@@
 		)
 		(property "Sheetname" "Z_ER_UP_AND_Z_ER_DOWN"
-			(at -34.29 43.7384 0)
+			(at -36.83 31.0384 0)
 			(effects
 				(font
@@
 		)
 		(property "Sheetfile" "z_er_up_and_z_er_dn.kicad_sch"
-			(at -34.29 61.5446 0)
+			(at -36.83 48.8446 0)
 			(effects
 				(font
@@
 				)
 			)
+		)
+	)
+	(sheet
+		(at -30.48 60.96)
+		(size 25.4 17.78)
+		(fields_autoplaced yes)
+		(stroke
+			(width 0.1524)
+			(type solid)
+		)
+		(fill
+			(color 0 0 0 0.0000)
+		)
+		(property "Sheetname" "VZB"
+			(at -30.48 60.2484 0)
+			(effects
+				(font
+					(size 1.27 1.27)
+				)
+				(justify left bottom)
+			)
+		)
+		(property "Sheetfile" "vzb.kicad_sch"
+			(at -30.48 79.3246 0)
+			(effects
+				(font
+					(size 1.27 1.27)
+				)
+				(justify left top)
+			)
+		)
+		(instances
+			(project "x_board"
+				(path "/5140f788-2f35-4c22-8e35-55ece5960fbd"
+					(page "4")
+				)
+			)

Commit message: Add Z PROTECTION circuit
Other:
- added sheet Z_PROTECTION (z_protection.kicad_sch)
Changed lines of the file:
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@@
 			(project "x_board"
 				(path "/5140f788-2f35-4c22-8e35-55ece5960fbd"
-					(page "2")
+					(page "3")
 				)
 			)
@@
 	)
 	(sheet
-		(at -36.83 31.75)
+		(at -36.83 60.96)
 		(size 24.13 16.51)
 		(fields_autoplaced yes)
@@
 		)
 		(property "Sheetname" "Z_ER_UP_AND_Z_ER_DOWN"
-			(at -36.83 31.0384 0)
+			(at -36.83 60.2484 0)
 			(effects
 				(font
@@
 		)
 		(property "Sheetfile" "z_er_up_and_z_er_dn.kicad_sch"
-			(at -36.83 48.8446 0)
-			(effects
-				(font
-					(size 1.27 1.27)
-				)
-				(justify left top)
-			)
-		)
-		(instances
-			(project "x_board"
-				(path "/5140f788-2f35-4c22-8e35-55ece5960fbd"
-					(page "3")
-				)
-			)
-		)
-	)
-	(sheet
-		(at -30.48 60.96)
-		(size 25.4 17.78)
-		(fields_autoplaced yes)
-		(stroke
-			(width 0.1524)
-			(type solid)
-		)
-		(fill
-			(color 0 0 0 0.0000)
-		)
-		(property "Sheetname" "VZB"
-			(at -30.48 60.2484 0)
-			(effects
-				(font
-					(size 1.27 1.27)
-				)
-				(justify left bottom)
-			)
-		)
-		(property "Sheetfile" "vzb.kicad_sch"
-			(at -30.48 79.3246 0)
+			(at -36.83 78.0546 0)
 			(effects
 				(font
@@
 				)
 			)
+		)
+	)
+	(sheet
+		(at -35.56 88.9)
+		(size 25.4 17.78)
+		(fields_autoplaced yes)
+		(stroke
+			(width 0.1524)
+			(type solid)
+		)
+		(fill
+			(color 0 0 0 0.0000)
+		)
+		(property "Sheetname" "VZB"
+			(at -35.56 88.1884 0)
+			(effects
+				(font
+					(size 1.27 1.27)
+				)
+				(justify left bottom)
+			)
+		)
+		(property "Sheetfile" "vzb.kicad_sch"
+			(at -35.56 107.2646 0)
+			(effects
+				(font
+					(size 1.27 1.27)
+				)
+				(justify left top)
+			)
+		)
+		(instances
+			(project "x_board"
+				(path "/5140f788-2f35-4c22-8e35-55ece5960fbd"
+					(page "5")
+				)
+			)
+		)
+	)
+	(sheet
+		(at -35.56 34.29)
+		(size 25.4 17.78)
+		(fields_autoplaced yes)
+		(stroke
+			(width 0.1524)
+			(type solid)
+		)
+		(fill
+			(color 0 0 0 0.0000)
+		)
+		(property "Sheetname" "Z_PROTECTION"
+			(at -35.56 33.5784 0)
+			(effects
+				(font
+					(size 1.27 1.27)
+				)
+				(justify left bottom)
+			)
+		)
+		(property "Sheetfile" "z_protection.kicad_sch"
+			(at -35.56 52.6546 0)
+			(effects
+				(font
+					(size 1.27 1.27)
+				)
+				(justify left top)
+			)
+		)
+		(instances
+			(project "x_board"
+				(path "/5140f788-2f35-4c22-8e35-55ece5960fbd"
+					(page "2")
+				)
+			)

Commit message: Add Z Control circuit
Other:
- added sheet Z_CONTROL (z_ctrl.kicad_sch)
Changed lines of the file:
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@@
 			(project "x_board"
 				(path "/5140f788-2f35-4c22-8e35-55ece5960fbd"
-					(page "5")
+					(page "6")
 				)
 			)
@@
 	)
 	(sheet
-		(at -36.83 60.96)
+		(at -35.56 100.33)
 		(size 24.13 16.51)
 		(fields_autoplaced yes)
@@
 		)
 		(property "Sheetname" "Z_ER_UP_AND_Z_ER_DOWN"
-			(at -36.83 60.2484 0)
+			(at -35.56 99.6184 0)
 			(effects
 				(font
@@
 		)
 		(property "Sheetfile" "z_er_up_and_z_er_dn.kicad_sch"
-			(at -36.83 78.0546 0)
+			(at -35.56 117.4246 0)
+			(effects
+				(font
+					(size 1.27 1.27)
+				)
+				(justify left top)
+			)
+		)
+		(instances
+			(project "x_board"
+				(path "/5140f788-2f35-4c22-8e35-55ece5960fbd"
+					(page "5")
+				)
+			)
+		)
+	)
+	(sheet
+		(at -34.29 128.27)
+		(size 25.4 17.78)
+		(fields_autoplaced yes)
+		(stroke
+			(width 0.1524)
+			(type solid)
+		)
+		(fill
+			(color 0 0 0 0.0000)
+		)
+		(property "Sheetname" "VZB"
+			(at -34.29 127.5584 0)
+			(effects
+				(font
+					(size 1.27 1.27)
+				)
+				(justify left bottom)
+			)
+		)
+		(property "Sheetfile" "vzb.kicad_sch"
+			(at -34.29 146.6346 0)
 			(effects
 				(font
@@
 	)
 	(sheet
-		(at -35.56 88.9)
+		(at -34.29 73.66)
 		(size 25.4 17.78)
 		(fields_autoplaced yes)
@@
 			(color 0 0 0 0.0000)
 		)
-		(property "Sheetname" "VZB"
-			(at -35.56 88.1884 0)
+		(property "Sheetname" "Z_PROTECTION"
+			(at -34.29 72.9484 0)
 			(effects
 				(font
@@
 			)
 		)
-		(property "Sheetfile" "vzb.kicad_sch"
-			(at -35.56 107.2646 0)
+		(property "Sheetfile" "z_protection.kicad_sch"
+			(at -34.29 92.0246 0)
 			(effects
 				(font
@@
 	)
 	(sheet
-		(at -35.56 34.29)
-		(size 25.4 17.78)
+		(at -34.29 40.64)
+		(size 22.86 13.97)
 		(fields_autoplaced yes)
 		(stroke
@@
 			(color 0 0 0 0.0000)
 		)
-		(property "Sheetname" "Z_PROTECTION"
-			(at -35.56 33.5784 0)
+		(property "Sheetname" "Z_CONTROL"
+			(at -34.29 39.9284 0)
 			(effects
 				(font
@@
 			)
 		)
-		(property "Sheetfile" "z_protection.kicad_sch"
-			(at -35.56 52.6546 0)
+		(property "Sheetfile" "z_ctrl.kicad_sch"
+			(at -34.29 55.1946 0)
 			(effects
 				(font

Commit message: Finishing implement X Board
Parts:
- removed C12, C13, C14: C_Small, symbol Device:C_Small
- removed C5: 1nF/1kV, symbol Device:C_Small
- removed D1: D_Filled, symbol Device:D_Filled
- removed FL28, FL29: L_Small, symbol Device:L_Small
- removed R13, R14: R_Small, symbol Device:R_Small
- added P2: Control Connection, symbol Connector:Conn_01x12_Pin
- added P3: Input Supply, symbol Connector:Conn_01x08_Pin
Connections:
- net 15V: now also P2.11 (Pin_11), P2.12 (Pin_12)
- net Earth: now also P2.8 (Pin_8), P2.9 (Pin_9), P3.4 (Pin_4), P3.5 (Pin_5)
- net VS_B: now also P3.7 (Pin_7), P3.8 (Pin_8)
- new net 5V: P2.10 (Pin_10)
- new net CTRL_OE: P2.7 (Pin_7)
- new net ER_CON: P3.1 (Pin_1), P3.2 (Pin_2)
- new net OE: P2.6 (Pin_6)
- new net Z_BIAS: P2.5 (Pin_5)
- new net Z_ER_DOWN: P2.4 (Pin_4)
- new net Z_ER_UP: P2.3 (Pin_3)
- new net Z_SUS_DOWN: P2.1 (Pin_1)
- new net Z_SUS_UP: P2.2 (Pin_2)
- no-connect marks 0 -> 2
Other:
- added sheet Z POWER SUPPLY (z_power_supply.kicad_sch)
- added sheet Z_OUT_CONNECTIONS (z_out_conn.kicad_sch)
- note added: "P2 1- Z_SUS_DN 2- Z_SUS_IP 3- Z_ER_UP 4- Z_ER_DN 5- Z_BIAS 6- OE 7- CTRL_OE 8- GND 9- GND 10- +5V 11- +15V 12- +15V"
- note added: "P3 1- ER_COM 2- ER_COM 3- NC 4- GND 5- GND 6- NC 7- +VS 8- +VS"

Commit message: Fix some Z-BOARD DRC
Other:
- note added: "INPUT CONNECTORS"
Changed lines of the file:
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@@
+		)
+	)
+	(text "INPUT CONNECTORS"
+		(exclude_from_sim no)
+		(at 154.94 20.32 0)
+		(effects
+			(font
+				(size 5 5)
+				(thickness 1)
+				(bold yes)
+				(italic yes)
+			)
 		)
 	)
@@
 		)
 	)
-	(label "INPUT CONNECTORS"
-		(at 196.85 27.94 180)
-		(effects
-			(font
-				(face "KiCad Font")
-				(size 5 5)
-				(thickness 0.254)
-				(bold yes)
-				(italic yes)
-			)
-			(justify right bottom)
-		)
-	)

Commit message: Finishing reverse engineering
Other:
- added sheet Measurements (P2) (measurements_p2.kicad_sch)
- added sheet Measurements (P3) (measurements_p3.kicad_sch)
- added sheet Measurements (P6 and P7) (measurements_p6_and_p7.kicad_sch)
Changed lines of the file:
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@@
+	)
+	(sheet
+		(at 300.99 25.4)
+		(size 22.86 13.97)
+		(fields_autoplaced yes)
+		(stroke
+			(width 0.1524)
+			(type solid)
+		)
+		(fill
+			(color 0 0 0 0.0000)
+		)
+		(property "Sheetname" "Measurements (P2)"
+			(at 300.99 24.6884 0)
+			(effects
+				(font
+					(size 1.27 1.27)
+				)
+				(justify left bottom)
+			)
+		)
+		(property "Sheetfile" "measurements_p2.kicad_sch"
+			(at 300.99 39.9546 0)
+			(effects
+				(font
+					(size 1.27 1.27)
+				)
+				(justify left top)
+			)
+		)
+		(instances
+			(project "x_board"
+				(path "/5140f788-2f35-4c22-8e35-55ece5960fbd"
+					(page "10")
+				)
+			)
+		)
 	)
 	(sheet
@@
 	)
 	(sheet
+		(at 302.26 54.61)
+		(size 22.86 13.97)
+		(fields_autoplaced yes)
+		(stroke
+			(width 0.1524)
+			(type solid)
+		)
+		(fill
+			(color 0 0 0 0.0000)
+		)
+		(property "Sheetname" "Measurements (P6 and P7)"
+			(at 302.26 53.8984 0)
+			(effects
+				(font
+					(size 1.27 1.27)
+				)
+				(justify left bottom)
+			)
+		)
+		(property "Sheetfile" "measurements_p6_and_p7.kicad_sch"
+			(at 302.26 69.1646 0)
+			(effects
+				(font
+					(size 1.27 1.27)
+				)
+				(justify left top)
+			)
+		)
+		(instances
+			(project "x_board"
+				(path "/5140f788-2f35-4c22-8e35-55ece5960fbd"
+					(page "11")
+				)
+			)
+		)
+	)
+	(sheet
 		(at -35.56 143.51)
 		(size 25.4 17.78)
@@
 				)
 			)
+		)
+	)
+	(sheet
+		(at 300.99 2.54)
+		(size 25.4 15.24)
+		(fields_autoplaced yes)
+		(stroke
+			(width 0.1524)
+			(type solid)
+		)
+		(fill
+			(color 0 0 0 0.0000)
+		)
+		(property "Sheetname" "Measurements (P3)"
+			(at 300.99 1.8284 0)
+			(effects
+				(font
+					(size 1.27 1.27)
+				)
+				(justify left bottom)
+			)
+		)
+		(property "Sheetfile" "measurements_p3.kicad_sch"
+			(at 300.99 18.3646 0)
+			(effects
+				(font
+					(size 1.27 1.27)
+				)
+				(justify left top)
+			)
+		)
+		(instances
+			(project "x_board"
+				(path "/5140f788-2f35-4c22-8e35-55ece5960fbd"
+					(page "9")
+				)
+			)
