File: TV_PLASMA/42PQ30R/x_board/vzb.kicad_sch (KiCad schematic)
At the start: 50 parts, among them Q1 Q_NMOS_GDS, Q2 Q_NMOS_GDS, Q3 Q_PNP_BCE, Q4 Q_PNP_BCE, Q51 Q_NMOS_GDS

Commit message: Correct VZB circuit
Connections:
- net at C11.2, C7.1, D7.2 (A)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: now also C3.2, C4.2, IC4.5 (GND)
Other:
- moved on the sheet: D8
Changed lines of the file:
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@@
+	)
+	(junction
+		(at 240.03 124.46)
+		(diameter 0)
+		(color 0 0 0 0)
 	)
 	(junction
@@
 	(junction
 		(at 167.64 130.81)
+		(diameter 0)
+		(color 0 0 0 0)
+	)
+	(junction
+		(at 261.62 92.71)
 		(diameter 0)
 		(color 0 0 0 0)
@@
 	(wire
 		(pts
+			(xy 186.69 99.06) (xy 223.52 99.06)
+		)
+		(stroke
+			(width 0)
+			(type default)
+		)
+	)
+	(wire
+		(pts
 			(xy 214.63 106.68) (xy 214.63 116.84)
 		)
@@
 	(wire
 		(pts
-			(xy 260.35 106.68) (xy 254 106.68)
-		)
-		(stroke
-			(width 0)
-			(type default)
-		)
-	)
-	(wire
-		(pts
 			(xy 158.75 68.58) (xy 161.29 68.58)
 		)
@@
 	(wire
 		(pts
-			(xy 260.35 99.06) (xy 260.35 106.68)
-		)
-		(stroke
-			(width 0)
-			(type default)
-		)
-	)
-	(wire
-		(pts
 			(xy 130.81 140.97) (xy 143.51 140.97)
 		)
@@
 	(wire
 		(pts
-			(xy 240.03 106.68) (xy 246.38 106.68)
-		)
-		(stroke
-			(width 0)
-			(type default)
-		)
-	)
-	(wire
-		(pts
 			(xy 161.29 92.71) (xy 173.99 92.71)
 		)
@@
 	(wire
 		(pts
+			(xy 261.62 124.46) (xy 261.62 92.71)
+		)
+		(stroke
+			(width 0)
+			(type default)
+		)
+	)
+	(wire
+		(pts
 			(xy 167.64 152.4) (xy 167.64 154.94)
 		)
@@
 	(wire
 		(pts
+			(xy 240.03 124.46) (xy 261.62 124.46)
+		)
+		(stroke
+			(width 0)
+			(type default)
+		)
+	)
+	(wire
+		(pts
 			(xy 107.95 109.22) (xy 107.95 115.57)
 		)
@@
 	(wire
 		(pts
+			(xy 240.03 99.06) (xy 240.03 106.68)
+		)
+		(stroke
+			(width 0)
+			(type default)
+		)
+	)
+	(wire
+		(pts
 			(xy 240.03 106.68) (xy 240.03 107.95)
 		)
@@
 	(wire
 		(pts
-			(xy 260.35 99.06) (xy 246.38 99.06)
+			(xy 231.14 99.06) (xy 240.03 99.06)
 		)
 		(stroke
@@
 	(global_label "15V_filter"
 		(shape input)
-		(at 246.38 99.06 180)
+		(at 186.69 99.06 180)
 		(fields_autoplaced yes)
 		(effects
@@
 		)
 		(property "Intersheetrefs" "${INTERSHEET_REFS}"
-			(at 234.3234 99.06 0)
+			(at 174.6334 99.06 0)
 			(effects
 				(font
@@
 	(symbol
 		(lib_id "Device:D_Filled")
-		(at 250.19 106.68 0)
-		(mirror x)
+		(at 227.33 99.06 0)
+		(mirror y)
 		(unit 1)
 		(exclude_from_sim no)
@@
 		(dnp no)
 		(property "Reference" "D8"
-			(at 250.19 102.87 0)
+			(at 227.33 96.52 0)
 			(effects
 				(font
@@
 		)
 		(property "Value" "D_Filled"
-			(at 250.19 110.49 0)
+			(at 227.33 95.25 0)
 			(effects
 				(font
@@
 		)
 		(property "Footprint" ""
-			(at 250.19 106.68 0)
+			(at 227.33 99.06 0)
 			(effects
 				(font
@@
 		)
 		(property "Datasheet" "~"
-			(at 250.19 106.68 0)
+			(at 227.33 99.06 0)
 			(effects
 				(font
@@
 		)
 		(property "Description" "Diode, filled shape"
-			(at 250.19 106.68 0)
+			(at 227.33 99.06 0)
 			(effects
 				(font
@@
 		)
 		(property "Sim.Device" "D"
-			(at 250.19 106.68 0)
+			(at 227.33 99.06 0)
 			(effects
 				(font
@@
 		)
 		(property "Sim.Pins" "1=K 2=A"
-			(at 250.19 106.68 0)
+			(at 227.33 99.06 0)
 			(effects
 				(font

Commit message: Finishing implement X Board
Parts:
- IC4: value ~ -> Unknown IC
Changed lines of the file:
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@@
 		(dnp no)
 		(property "Reference" "IC4"
-			(at 187.96 110.49 0)
+			(at 187.96 109.22 0)
 			(effects
 				(font
@@
 			)
 		)
-		(property "Value" "~"
+		(property "Value" "Unknown IC"
 			(at 187.96 111.76 0)
 			(effects

Commit message: Fix some Z-BOARD DRC
Parts:
- R278, R279: value 470k -> 47k
- R46: renamed from R18; value 470k -> 47k
- R47: renamed from R17; value 470k -> 47k
- renumbered C144 to C149
Other:
- note added: "VZB"
Changed lines of the file:
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@@
 		)
 	)
-	(label "VZB"
-		(at 146.05 24.13 180)
+	(text "VZB"
+		(exclude_from_sim no)
+		(at 142.24 21.59 0)
 		(effects
 			(font
-				(face "KiCad Font")
 				(size 5 5)
 				(thickness 0.254)
@@
 				(italic yes)
 			)
-			(justify right bottom)
 		)
 	)
@@
 		(on_board yes)
 		(dnp no)
-		(property "Reference" "C144"
+		(property "Reference" "C149"
 			(at 87.63 104.14 0)
 			(effects
@@
 			(project "x_board"
 				(path "/5140f788-2f35-4c22-8e35-55ece5960fbd/5833f712-63ee-492f-b888-d285859535d4"
-					(reference "C144")
+					(reference "C149")
 					(unit 1)
 				)
@@
 			)
 		)
-		(property "Value" "470k"
+		(property "Value" "47k"
 			(at 104.14 63.5 0)
 			(effects
@@
 		(dnp no)
 		(property "Reference" "VR8"
-			(at 100.33 88.9 0)
+			(at 111.76 82.55 0)
 			(effects
 				(font
@@
 		)
 		(property "Value" "100K"
-			(at 101.6 91.44 0)
+			(at 111.76 85.09 0)
 			(effects
 				(font
@@
 			)
 		)
-		(property "Value" "470k"
+		(property "Value" "47k"
 			(at 104.14 73.66 0)
 			(effects
@@
 		(on_board yes)
 		(dnp no)
-		(property "Reference" "R18"
+		(property "Reference" "R46"
 			(at 104.14 106.68 0)
 			(effects
@@
 			)
 		)
-		(property "Value" "470k"
+		(property "Value" "47k"
 			(at 104.14 109.22 0)
 			(effects
@@
 			(project "x_board"
 				(path "/5140f788-2f35-4c22-8e35-55ece5960fbd/5833f712-63ee-492f-b888-d285859535d4"
-					(reference "R18")
+					(reference "R46")
 					(unit 1)
 				)
@@
 		(on_board yes)
 		(dnp no)
-		(property "Reference" "R17"
+		(property "Reference" "R47"
 			(at 104.14 96.52 0)
 			(effects
@@
 			)
 		)
-		(property "Value" "470k"
+		(property "Value" "47k"
 			(at 104.14 99.06 0)
 			(effects
@@
 			(project "x_board"
 				(path "/5140f788-2f35-4c22-8e35-55ece5960fbd/5833f712-63ee-492f-b888-d285859535d4"
-					(reference "R17")
+					(reference "R47")
 					(unit 1)
 				)

Commit message: Update C3, C7 and C168 Capacitances values in Z Board
Parts:
- C168, C3: value C_Small -> 1uF
- C7: value C_Small -> 100nF
Changed lines of the file:
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@@
 			)
 		)
-		(property "Value" "C_Small"
-			(at 163.83 101.6062 0)
+		(property "Value" "100nF"
+			(at 153.67 101.6 0)
 			(effects
 				(font
@@
 				)
 				(justify left)
-				(hide yes)
 			)
 		)
@@
 		(dnp no)
 		(property "Reference" "C3"
-			(at 224.79 118.11 0)
+			(at 218.44 113.03 0)
 			(effects
 				(font
@@
 			)
 		)
-		(property "Value" "C_Small"
-			(at 224.79 116.8462 0)
+		(property "Value" "1uF"
+			(at 217.17 116.84 0)
 			(effects
 				(font
@@
 				)
 				(justify left)
-				(hide yes)
 			)
 		)
@@
 		(dnp no)
 		(property "Reference" "C168"
-			(at 142.24 127 0)
+			(at 142.24 121.92 0)
 			(effects
 				(font
@@
 			)
 		)
-		(property "Value" "C_Small"
-			(at 152.4 125.7362 0)
+		(property "Value" "1uF"
+			(at 142.24 125.73 0)
 			(effects
 				(font
@@
 				)
 				(justify left)
-				(hide yes)
-			)
-		)
+			)
+		)

Commit message: Add capacitors value, rename correct resistor
Parts:
- C11: value C_Small -> 127nF
- C149: value C_Small -> 100nF
- C4: value C_Small -> 47uF/25V
- C6: value C_Small -> 470 nF
- renumbered D8 to D2
Changed lines of the file:
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@@
 		(on_board yes)
 		(dnp no)
-		(property "Reference" "D8"
+		(property "Reference" "D2"
 			(at 227.33 96.52 0)
 			(effects
@@
 			(project "x_board"
 				(path "/5140f788-2f35-4c22-8e35-55ece5960fbd/5833f712-63ee-492f-b888-d285859535d4"
-					(reference "D8")
+					(reference "D2")
 					(unit 1)
 				)
@@
 		(dnp no)
 		(property "Reference" "C149"
-			(at 87.63 104.14 0)
-			(effects
-				(font
-					(size 1.27 1.27)
-				)
-				(justify left)
-			)
-		)
-		(property "Value" "C_Small"
-			(at 96.52 102.8762 0)
-			(effects
-				(font
-					(size 1.27 1.27)
-				)
-				(justify left)
-				(hide yes)
+			(at 85.09 100.33 0)
+			(effects
+				(font
+					(size 1.27 1.27)
+				)
+				(justify left)
+			)
+		)
+		(property "Value" "100nF"
+			(at 85.09 102.87 0)
+			(effects
+				(font
+					(size 1.27 1.27)
+				)
+				(justify left)
 			)
 		)
@@
 		(dnp no)
 		(property "Reference" "C11"
-			(at 256.54 77.47 0)
-			(effects
-				(font
-					(size 1.27 1.27)
-				)
-				(justify left)
-			)
-		)
-		(property "Value" "C_Small"
+			(at 264.16 76.2 0)
+			(effects
+				(font
+					(size 1.27 1.27)
+				)
+				(justify left)
+			)
+		)
+		(property "Value" "127nF"
 			(at 264.16 80.0162 0)
 			(effects
@@
 				)
 				(justify left)
-				(hide yes)
 			)
 		)
@@
 			)
 		)
-		(property "Value" "C_Small"
-			(at 184.15 62.2362 0)
-			(effects
-				(font
-					(size 1.27 1.27)
-				)
-				(justify left)
-				(hide yes)
+		(property "Value" "470 nF"
+			(at 171.45 62.23 0)
+			(effects
+				(font
+					(size 1.27 1.27)
+				)
+				(justify left)
 			)
 		)
@@
 		(dnp no)
 		(property "Reference" "C4"
-			(at 234.95 118.11 0)
-			(effects
-				(font
-					(size 1.27 1.27)
-				)
-				(justify left)
-			)
-		)
-		(property "Value" "C_Small"
+			(at 242.57 118.11 0)
+			(effects
+				(font
+					(size 1.27 1.27)
+				)
+				(justify left)
+			)
+		)
+		(property "Value" "47uF/25V"
 			(at 242.57 120.6562 0)
 			(effects
@@
 				)
 				(justify left)
-				(hide yes)
-			)
-		)
+			)
+		)

Commit message: Modify optocouple "Unknown IC" after test
Parts:
- removed Q3: Q_PNP_BCE, symbol Device:Q_PNP_BCE
- added Q3: Q_NMOS_GDS, Package_TO_SOT_SMD:TO-252-2, symbol Device:Q_NMOS_GDS
Connections:
- net Earth: now also Q3.3 (S)
- net at R37.2: now also Q3.1 (G)
- net at IC4.3 (K), R38.2: now also Q3.2 (D)
Changed lines of the file:
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@@
 	)
 	(junction
-		(at 167.64 152.4)
-		(diameter 0)
-		(color 0 0 0 0)
-	)
-	(junction
 		(at 240.03 124.46)
 		(diameter 0)
@@
 	)
 	(junction
+		(at 167.64 152.4)
+		(diameter 0)
+		(color 0 0 0 0)
+	)
+	(junction
 		(at 173.99 92.71)
 		(diameter 0)
@@
 	)
 	(symbol
-		(lib_id "Device:R_Small")
-		(at 64.77 71.12 180)
+		(lib_name "3411918_1")
+		(lib_id "irf_s21850:3411918")
+		(at 187.96 113.03 0)
 		(unit 1)
 		(exclude_from_sim no)
@@
 		(on_board yes)
 		(dnp no)
-		(property "Reference" "R42"
-			(at 60.96 71.12 0)
+		(fields_autoplaced yes)
+		(property "Reference" "IC4"
+			(at 187.96 109.22 0)
 			(effects
 				(font
@@
 			)
 		)
-		(property "Value" "22"
-			(at 62.23 73.66 0)
+		(property "Value" "Unknown IC"
+			(at 187.96 111.76 0)
 			(effects
 				(font
 					(size 1.27 1.27)
 				)
-				(justify bottom)
 			)
 		)
 		(property "Footprint" ""
-			(at 64.77 71.12 0)
+			(at 187.96 113.03 0)
 			(effects
 				(font
@@
 			)
 		)
-		(property "Datasheet" "~"
-			(at 64.77 71.12 0)
+		(property "Datasheet" ""
+			(at 187.96 113.03 0)
 			(effects
 				(font
@@
 			)
 		)
-		(property "Description" "Resistor, small symbol"
-			(at 64.77 71.12 0)
+		(property "Description" ""
+			(at 187.96 113.03 0)
 			(effects
 				(font
@@
 			)
 		)
-		(pin "1"
+		(pin "8"
+		)
+		(pin "6"
 		)
 		(pin "2"
 		)
+		(pin "1"
+		)
+		(pin "5"
+		)
+		(pin "3"
+		)
+		(pin "7"
+		)
+		(pin "4"
+		)
 		(instances
-			(project "x_board"
+			(project ""
 				(path "/5140f788-2f35-4c22-8e35-55ece5960fbd/5833f712-63ee-492f-b888-d285859535d4"
-					(reference "R42")
+					(reference "IC4")
 					(unit 1)
 				)
@@
 	)
 	(symbol
-		(lib_id "irf_s21850:3411918")
-		(at 187.96 113.03 0)
+		(lib_id "Device:R_Small")
+		(at 64.77 71.12 180)
 		(unit 1)
 		(exclude_from_sim no)
@@
 		(on_board yes)
 		(dnp no)
-		(property "Reference" "IC4"
-			(at 187.96 109.22 0)
+		(property "Reference" "R42"
+			(at 60.96 71.12 0)
 			(effects
 				(font
@@
 			)
 		)
-		(property "Value" "Unknown IC"
-			(at 187.96 111.76 0)
+		(property "Value" "22"
+			(at 62.23 73.66 0)
 			(effects
 				(font
 					(size 1.27 1.27)
 				)
+				(justify bottom)
 			)
 		)
 		(property "Footprint" ""
-			(at 187.96 113.03 0)
+			(at 64.77 71.12 0)
 			(effects
 				(font
@@
 			)
 		)
-		(property "Datasheet" ""
-			(at 187.96 113.03 0)
+		(property "Datasheet" "~"
+			(at 64.77 71.12 0)
 			(effects
 				(font
@@
 			)
 		)
-		(property "Description" ""
-			(at 187.96 113.03 0)
+		(property "Description" "Resistor, small symbol"
+			(at 64.77 71.12 0)
 			(effects
 				(font
@@
 			)
 		)
-		(pin "3"
-		)
-		(pin "7"
+		(pin "1"
 		)
 		(pin "2"
 		)
-		(pin "8"
-		)
-		(pin "4"
-		)
-		(pin "5"
-		)
-		(pin "6"
-		)
-		(pin "1"
-		)
 		(instances
-			(project ""
+			(project "x_board"
 				(path "/5140f788-2f35-4c22-8e35-55ece5960fbd/5833f712-63ee-492f-b888-d285859535d4"
-					(reference "IC4")
+					(reference "R42")
 					(unit 1)
 				)
@@
 	)
 	(symbol
+		(lib_id "Device:Q_NMOS_GDS")
+		(at 165.1 140.97 0)
+		(unit 1)
+		(exclude_from_sim no)
+		(in_bom yes)
+		(on_board yes)
+		(dnp no)
+		(property "Reference" "Q3"
+			(at 171.45 139.6999 0)
+			(effects
+				(font
+					(size 1.27 1.27)
+				)
+				(justify left)
+			)
+		)
+		(property "Value" "Q_NMOS_GDS"
+			(at 171.45 142.2399 0)
+			(effects
+				(font
+					(size 1.27 1.27)
+				)
+				(justify left)
+				(hide yes)
+			)
+		)
+		(property "Footprint" "Package_TO_SOT_SMD:TO-252-2"
+			(at 170.18 138.43 0)
+			(effects
+				(font
+					(size 1.27 1.27)
+				)
+				(hide yes)
+			)
+		)
+		(property "Datasheet" "~"
+			(at 165.1 140.97 0)
+			(effects
+				(font
+					(size 1.27 1.27)
+				)
+				(hide yes)
+			)
+		)
+		(property "Description" "N-MOSFET transistor, gate/drain/source"
+			(at 165.1 140.97 0)
+			(effects
+				(font
+					(size 1.27 1.27)
+				)
+				(hide yes)
+			)
+		)
+		(pin "3"
+		)
+		(pin "1"
+		)
+		(pin "2"
+		)
+		(instances
+			(project "x_board"
+				(path "/5140f788-2f35-4c22-8e35-55ece5960fbd/5833f712-63ee-492f-b888-d285859535d4"
+					(reference "Q3")
+					(unit 1)
+				)
+			)
+		)
+	)
+	(symbol
 		(lib_id "Device:R_Small")
 		(at 107.95 60.96 180)
@@
 					(unit 1)
 				)
-			)
-		)
-	)
-	(symbol
-		(lib_id "Device:Q_PNP_BCE")
-		(at 165.1 140.97 0)
-		(mirror x)
-		(unit 1)
-		(exclude_from_sim no)
-		(in_bom yes)
-		(on_board yes)
-		(dnp no)
-		(property "Reference" "Q3"
-			(at 170.18 139.6999 0)
-			(effects
-				(font
-					(size 1.27 1.27)
-				)
-				(justify left)
-			)
-		)
-		(property "Value" "Q_PNP_BCE"
-			(at 170.18 142.2399 0)
-			(effects
-				(font
-					(size 1.27 1.27)
-				)
-				(justify left)
-				(hide yes)
-			)
-		)
-		(property "Footprint" ""
-			(at 170.18 143.51 0)
-			(effects
-				(font
-					(size 1.27 1.27)
-				)
-				(hide yes)
-			)
-		)
-		(property "Datasheet" "~"
-			(at 165.1 140.97 0)
-			(effects
-				(font
-					(size 1.27 1.27)
-				)
-				(hide yes)
-			)
-		)
-		(property "Description" "PNP transistor, base/collector/emitter"
-			(at 165.1 140.97 0)
-			(effects
-				(font
-					(size 1.27 1.27)
-				)
-				(hide yes)
-			)
-		)
-		(pin "3"
-		)
-		(pin "1"
-		)
-		(pin "2"
-		)
-		(instances
-			(project "x_board"
-				(path "/5140f788-2f35-4c22-8e35-55ece5960fbd/5833f712-63ee-492f-b888-d285859535d4"
-					(reference "Q3")
-					(unit 1)
-				)

Commit message: Adding Z board top detailed
Parts:
- C159: value C_Small -> 1uF / 500V
Other:
- moved on the sheet: C159
Changed lines of the file:
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@@
 	(wire
 		(pts
-			(xy 57.15 106.68) (xy 57.15 107.95)
+			(xy 57.15 106.68) (xy 57.15 109.22)
 		)
 		(stroke
@@
 	(wire
 		(pts
-			(xy 57.15 113.03) (xy 57.15 127)
+			(xy 57.15 114.3) (xy 57.15 127)
 		)
 		(stroke
@@
 	(symbol
 		(lib_id "Device:C_Small")
-		(at 57.15 110.49 0)
+		(at 57.15 111.76 0)
 		(unit 1)
 		(exclude_from_sim no)
@@
 		(dnp no)
 		(property "Reference" "C159"
-			(at 49.53 111.76 0)
+			(at 49.53 113.03 0)
 			(effects
 				(font
@@
 			)
 		)
-		(property "Value" "C_Small"
-			(at 59.69 111.7662 0)
+		(property "Value" "1uF / 500V"
+			(at 44.45 115.57 0)
 			(effects
 				(font
@@
 				)
 				(justify left)
-				(hide yes)
 			)
 		)
 		(property "Footprint" ""
-			(at 57.15 110.49 0)
+			(at 57.15 111.76 0)
 			(effects
 				(font
@@
 		)
 		(property "Datasheet" "~"
-			(at 57.15 110.49 0)
+			(at 57.15 111.76 0)
 			(effects
 				(font
@@
 		)
 		(property "Description" "Unpolarized capacitor, small symbol"
-			(at 57.15 110.49 0)
-			(effects
-				(font
+			(at 57.15 111.76 0)
+			(effects
+				(font
