File: TV_PLASMA/42PQ30R/x_board/z_power_supply.kicad_sch (KiCad schematic)
At the start: 9 parts

Commit message: Fix some Z-BOARD DRC
Parts:
- renumbered C2 to C12, C5 to C13, C12 to C14, C1 to C5
Other:
- note added: "Z POWER SUPPLY"
Changed lines of the file:
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@@
 		)
 	)
-	(label "Z POWER SUPPLY"
-		(at 175.26 29.21 180)
+	(text "Z POWER SUPPLY"
+		(exclude_from_sim no)
+		(at 143.51 26.67 0)
 		(effects
 			(font
-				(face "KiCad Font")
 				(size 5 5)
-				(thickness 0.254)
+				(thickness 1)
 				(bold yes)
 				(italic yes)
 			)
-			(justify right bottom)
 		)
 	)
@@
 		(dnp no)
 		(fields_autoplaced yes)
-		(property "Reference" "C12"
+		(property "Reference" "C14"
 			(at 171.45 88.9062 0)
 			(effects
@@
 			(project "x_board"
 				(path "/5140f788-2f35-4c22-8e35-55ece5960fbd/4b9b2cd4-424c-4bdb-b6b4-ab40bea37f9b"
-					(reference "C12")
+					(reference "C14")
 					(unit 1)
 				)
@@
 		(on_board yes)
 		(dnp no)
-		(property "Reference" "C1"
+		(property "Reference" "C5"
 			(at 137.16 88.9062 0)
 			(effects
@@
 			(project "x_board"
 				(path "/5140f788-2f35-4c22-8e35-55ece5960fbd/4b9b2cd4-424c-4bdb-b6b4-ab40bea37f9b"
-					(reference "C1")
+					(reference "C5")
 					(unit 1)
 				)
@@
 		(dnp no)
 		(fields_autoplaced yes)
-		(property "Reference" "C2"
+		(property "Reference" "C12"
 			(at 152.4 88.9062 0)
 			(effects
@@
 			(project "x_board"
 				(path "/5140f788-2f35-4c22-8e35-55ece5960fbd/4b9b2cd4-424c-4bdb-b6b4-ab40bea37f9b"
-					(reference "C2")
+					(reference "C12")
 					(unit 1)
 				)
@@
 		(dnp no)
 		(fields_autoplaced yes)
-		(property "Reference" "C5"
+		(property "Reference" "C13"
 			(at 162.56 88.9062 0)
 			(effects
@@
 			(project "x_board"
 				(path "/5140f788-2f35-4c22-8e35-55ece5960fbd/4b9b2cd4-424c-4bdb-b6b4-ab40bea37f9b"
-					(reference "C5")
-					(unit 1)
-				)
+					(reference "C13")
+					(unit 1)
+				)

Commit message: Adding Z board top detailed
Parts:
- C12, C13, C14: value C_Small -> 3.3uF/250V
- R13, R14: value R_Small -> 1R
Other:
- moved on the sheet: C13, C14, D1, R14
